Commit message: Update urdf

File: lunabotics_sim_v1_description/urdf/lunabotics_sim_v1_description.urdf (robot description, URDF)
Before this commit: robot lunabotics_sim_v1_description, 5 links, 4 joints
Joints:
- joint wheel_1: origin xyz=0.56598 -0.58121 0.40454 rpy=1.5708 0.39309 -3.1416 -> xyz=0.2788 0.15558 0.97581 rpy=3.1416 0 -2.7485
- joint wheel_2: origin xyz=-0.043122 -0.58121 0.40454 rpy=1.5708 0 0 -> xyz=-0.3303 0.15558 0.97581 rpy=0 0 0
- joint wheel_3: origin xyz=0.56598 -0.97811 0.40454 rpy=1.5708 0 0 -> xyz=0.2788 0.15558 1.3727 rpy=0 0 0
- joint wheel_4: origin xyz=-0.043122 -0.97811 0.40454 rpy=-1.5708 -0.50649 3.1416 -> xyz=-0.3303 0.15558 1.3727 rpy=0 0 2.6351
