Commit message: fixed urdf and simulation code

File: dummy_bot_description/urdf/dummy_bot.xacro (robot description, xacro)
@@ -1,4 +1,24 @@
 <?xml version="1.0" ?>
 <robot name="dummy_bot" xmlns:xacro="http://www.ros.org/wiki/xacro">
+<xacro:property name="PI" value="3.1415926535897931"/>
+<xacro:property name="chassisHeight" value="0.2"/>
+<xacro:property name="chassisLength" value="1.0"/>
+<xacro:property name="chassisWidth" value="0.5"/>
+<xacro:property name="chassisMass" value="50"/>
+<xacro:property name="wheelWidth" value="0.05"/>
+<xacro:property name="wheelRadius" value="0.2"/>
+<xacro:property name="wheelMass" value="5"/>
+<xacro:macro name="box_inertia" params="m x y z">
+  <inertia  ixx="${m*(y*y+z*z)/12}" ixy = "0" ixz = "0"
+    iyy="${m*(x*x+z*z)/12}" iyz = "0"
+    izz="${m*(x*x+z*z)/12}"
+  />
+</xacro:macro>
+<xacro:macro name="cylinder_inertia" params="m r h">
+  <inertia  ixx="${m*(3*r*r+h*h)/12}" ixy = "0" ixz = "0"
+    iyy="${m*(3*r*r+h*h)/12}" iyz = "0"
+    izz="${m*r*r/2}"
+  />
+</xacro:macro>
 <xacro:include filename="$(find dummy_bot_description)/urdf/materials.xacro" />
 <xacro:include filename="$(find dummy_bot_description)/urdf/dummy_bot.trans" />
@@ -6,7 +26,7 @@
 <link name="base_link">
   <inertial>
-    <origin rpy="0 0 0" xyz="-1.667754803659369e-10 0.0 0.08835894305363262"/>
-    <mass value="369.7501727616167"/>
-    <inertia ixx="8.465112" ixy="0.0" ixz="0.0" iyy="18.141277" iyz="0.0" izz="25.579367"/>
+    <origin rpy="0 0 0" xyz="0 0.0 0.08835894305363262"/>
+    <mass value="${chassisMass}"/>
+    <xacro:box_inertia m="${chassisMass}" x="1" y="0.5" z="0.15"/>
   </inertial>
   <visual>
@@ -24,14 +44,14 @@
   </collision>
 </link>
-<link name="wheel_right_front_1">
+<link name="right_front">
   <inertial>
     <origin rpy="0 0 0" xyz="-4.3576253716537394e-14 -0.022224999999999995 -2.736260904245835e-07"/>
-    <mass value="43.1518870370614"/>
-    <inertia ixx="0.445692" ixy="0.0" ixz="0.0" iyy="0.877173" iyz="0.0" izz="0.445692"/>
+    <mass value="${wheelMass}"/>
+    <xacro:cylinder_inertia m="${wheelMass}" r="${wheelRadius}" h="${wheelWidth}"/>
   </inertial>
   <visual>
     <origin rpy="0 0 0" xyz="-0.254 0.254 -0.101276"/>
     <geometry>
-      <mesh filename="package://dummy_bot_description/meshes/wheel_right_front_1.stl" scale="0.001 0.001 0.001"/>
+      <mesh filename="package://dummy_bot_description/meshes/right_front.stl" scale="0.001 0.001 0.001"/>
     </geometry>
     <material name="silver"/>
@@ -40,18 +60,18 @@
     <origin rpy="0 0 0" xyz="-0.254 0.254 -0.101276"/>
     <geometry>
-      <mesh filename="package://dummy_bot_description/meshes/wheel_right_front_1.stl" scale="0.001 0.001 0.001"/>
+      <mesh filename="package://dummy_bot_description/meshes/right_front.stl" scale="0.001 0.001 0.001"/>
     </geometry>
   </collision>
 </link>
-<link name="wheel_1_left_front_1">
+<link name="left_front">
   <inertial>
     <origin rpy="0 0 0" xyz="-4.3576253716537394e-14 0.02222499999999994 -2.736260904245835e-07"/>
-    <mass value="43.1518870370614"/>
-    <inertia ixx="0.445692" ixy="-0.0" ixz="0.0" iyy="0.877173" iyz="0.0" izz="0.445692"/>
+    <mass value="${wheelMass}"/>
+    <xacro:cylinder_inertia m="${wheelMass}" r="${wheelRadius}" h="${wheelWidth}"/>
   </inertial>
   <visual>
     <origin rpy="0 0 0" xyz="-0.254 -0.254 -0.101276"/>
     <geometry>
-      <mesh filename="package://dummy_bot_description/meshes/wheel_1_left_front_1.stl" scale="0.001 0.001 0.001"/>
+      <mesh filename="package://dummy_bot_description/meshes/left_front.stl" scale="0.001 0.001 0.001"/>
     </geometry>
     <material name="silver"/>
@@ -60,18 +80,18 @@
     <origin rpy="0 0 0" xyz="-0.254 -0.254 -0.101276"/>
     <geometry>
-      <mesh filename="package://dummy_bot_description/meshes/wheel_1_left_front_1.stl" scale="0.001 0.001 0.001"/>
+      <mesh filename="package://dummy_bot_description/meshes/left_front.stl" scale="0.001 0.001 0.001"/>
     </geometry>
   </collision>
 </link>
-<link name="wheel_left_back_1">
+<link name="left_back">
   <inertial>
     <origin rpy="0 0 0" xyz="-4.346523141407488e-14 0.02222499999999994 -2.7362609036907237e-07"/>
-    <mass value="43.1518870370614"/>
-    <inertia ixx="0.445692" ixy="-0.0" ixz="0.0" iyy="0.877173" iyz="0.0" izz="0.445692"/>
+    <mass value="${wheelMass}"/>
+    <xacro:cylinder_inertia m="${wheelMass}" r="${wheelRadius}" h="${wheelWidth}"/>
   </inertial>
   <visual>
     <origin rpy="0 0 0" xyz="0.254 -0.254 -0.101276"/>
     <geometry>
-      <mesh filename="package://dummy_bot_description/meshes/wheel_left_back_1.stl" scale="0.001 0.001 0.001"/>
+      <mesh filename="package://dummy_bot_description/meshes/left_back.stl" scale="0.001 0.001 0.001"/>
     </geometry>
     <material name="silver"/>
@@ -80,18 +100,18 @@
     <origin rpy="0 0 0" xyz="0.254 -0.254 -0.101276"/>
     <geometry>
-      <mesh filename="package://dummy_bot_description/meshes/wheel_left_back_1.stl" scale="0.001 0.001 0.001"/>
+      <mesh filename="package://dummy_bot_description/meshes/left_back.stl" scale="0.001 0.001 0.001"/>
     </geometry>
   </collision>
 </link>
-<link name="wheel_right_back_1">
+<link name="right_back">
   <inertial>
     <origin rpy="0 0 0" xyz="-4.3520742565306136e-14 -0.022224999999999995 -2.736260904245835e-07"/>
-    <mass value="43.1518870370614"/>
-    <inertia ixx="0.445692" ixy="-0.0" ixz="0.0" iyy="0.877173" iyz="0.0" izz="0.445692"/>
+    <mass value="${wheelMass}"/>
+    <xacro:cylinder_inertia m="${wheelMass}" r="${wheelRadius}" h="${wheelWidth}"/>
   </inertial>
   <visual>
     <origin rpy="0 0 0" xyz="0.254 0.254 -0.101276"/>
     <geometry>
-      <mesh filename="package://dummy_bot_description/meshes/wheel_right_back_1.stl" scale="0.001 0.001 0.001"/>
+      <mesh filename="package://dummy_bot_description/meshes/right_back.stl" scale="0.001 0.001 0.001"/>
     </geometry>
     <material name="silver"/>
@@ -100,31 +120,38 @@
     <origin rpy="0 0 0" xyz="0.254 0.254 -0.101276"/>
     <geometry>
-      <mesh filename="package://dummy_bot_description/meshes/wheel_right_back_1.stl" scale="0.001 0.001 0.001"/>
+      <mesh filename="package://dummy_bot_description/meshes/right_back.stl" scale="0.001 0.001 0.001"/>
     </geometry>
   </collision>
 </link>
-<joint name="Rev1" type="continuous">
+<joint name="right_front_rev" type="continuous">
   <origin rpy="0 0 0" xyz="0.254 -0.254 0.101276"/>
   <parent link="base_link"/>
-  <child link="wheel_right_front_1"/>
+  <child link="right_front"/>
   <axis xyz="0.0 1.0 0.0"/>
 </joint>
-<joint name="Rev2" type="continuous">
+<joint name="left_front_rev" type="continuous">
   <origin rpy="0 0 0" xyz="0.254 0.254 0.101276"/>
   <parent link="base_link"/>
-  <child link="wheel_1_left_front_1"/>
+  <child link="left_front"/>
   <axis xyz="0.0 -1.0 0.0"/>
 </joint>
-<joint name="Rev3" type="continuous">
+<joint name="left_back_rev" type="continuous">
   <origin rpy="0 0 0" xyz="-0.254 0.254 0.101276"/>
   <parent link="base_link"/>
-  <child link="wheel_left_back_1"/>
+  <child link="left_back"/>
   <axis xyz="0.0 -1.0 0.0"/>
 </joint>
-<joint name="Rev4" type="continuous">
+<joint name="right_back_rev" type="continuous">
   <origin rpy="0 0 0" xyz="-0.254 -0.254 0.101276"/>
   <parent link="base_link"/>
-  <child link="wheel_right_back_1"/>
+  <child link="right_back"/>
   <axis xyz="0.0 1.0 0.0"/>
 </joint>
+<xacro:include filename="$(find realsense_ros_gazebo)/xacro/depthcam.xacro"/>
+<xacro:realsense_d435 sensor_name="d435_cam_forward" parent_link="base_link" rate="10">
+  <origin xyz="0.000 0.229 0.482" rpy="0 0 0" />
+</xacro:realsense_d435>
+<xacro:realsense_d435 sensor_name="d435_cam_backward" parent_link="base_link" rate="10">
+  <origin xyz="0.000 0.20 0.482" rpy="0 0 3.1415" />
+</xacro:realsense_d435>
 </robot>
