Commit message: Sim fixes

File: lunabot_sim/dummy_bot_description/urdf/dummy_bot.xacro (robot description, xacro)
@@ -2,6 +2,6 @@
 <robot name="dummy_bot" xmlns:xacro="http://www.ros.org/wiki/xacro">
 <xacro:property name="PI" value="3.1415926535897931"/>
-<xacro:property name="chassisHeight" value="0.2"/>
-<xacro:property name="chassisLength" value="1.0"/>
+<xacro:property name="chassisHeight" value="0.1"/>
+<xacro:property name="chassisLength" value="0.8"/>
 <xacro:property name="chassisWidth" value="0.5"/>
 <xacro:property name="chassisMass" value="50"/>
@@ -28,5 +28,5 @@
     <origin rpy="0 0 0" xyz="0 0.0 0.08835894305363262"/>
     <mass value="${chassisMass}"/>
-    <xacro:box_inertia m="${chassisMass}" x="1" y="0.5" z="0.15"/>
+    <xacro:box_inertia m="${chassisMass}" x="${chassisLength}" y="${chassisWidth}" z="${chassisHeight}"/>
   </inertial>
   <visual>
