Commit message: computer updates

File: lunabot_sim/lunabot_description/urdf/lunabot.xacro (robot description, xacro)
@@ -148,9 +148,9 @@
   <axis xyz="0.0 1.0 0.0"/>
 </joint>
-<link name="d455_front_color_optical_frame"/>
+<link name="d455_back_link"/>
 <joint name="depth_cam_jnt" type="fixed">
-    <origin rpy="${-PI/2} 0 ${PI/2}" xyz="-0.457877 0.188509 0.255037"/>
+    <origin rpy="-2.0000019999706227e-06 0.0019999983333319994 3.139592651256459" xyz="-0.457877 0.129509 0.255037"/>
   <parent link="base_link"/>
-  <child link="d455_front_color_optical_frame"/>
+  <child link="d455_back_link"/>
   <axis xyz="0.0 1.0 0.0"/>
 </joint>

Commit message: fixed robot sim positions

File: lunabot_sim/lunabot_description/urdf/lunabot.xacro (robot description, xacro)
@@ -3,9 +3,9 @@
 <xacro:property name="PI" value="3.1415926535897931"/>
 <xacro:property name="chassisHeight" value="0.2"/>
-<xacro:property name="chassisLength" value="1.0"/>
+<xacro:property name="chassisLength" value="0.82"/>
 <xacro:property name="chassisWidth" value="0.5"/>
-<xacro:property name="chassisMass" value="50"/>
+<xacro:property name="chassisMass" value="55"/>
 <xacro:property name="wheelWidth" value="0.05"/>
-<xacro:property name="wheelRadius" value="0.2"/>
+<xacro:property name="wheelRadius" value="0.13755"/>
 <xacro:property name="wheelMass" value="5"/>
 <xacro:macro name="box_inertia" params="m x y z">
@@ -40,5 +40,5 @@
 <link name="right_front">
   <inertial>
-    <origin rpy="0 0 0" xyz="-4.3576253716537394e-14 -0.022224999999999995 -2.736260904245835e-07"/>
+    <origin rpy="0 0 0" xyz="0 0 0"/>
     <mass value="${wheelMass}"/>
     <xacro:cylinder_inertia m="${wheelMass}" r="${wheelRadius}" h="${wheelWidth}"/>
@@ -60,5 +60,5 @@
 <link name="left_front">
   <inertial>
-    <origin rpy="0 0 0" xyz="-4.3576253716537394e-14 0.02222499999999994 -2.736260904245835e-07"/>
+    <origin rpy="0 0 0" xyz="0 0 0"/>
     <mass value="${wheelMass}"/>
     <xacro:cylinder_inertia m="${wheelMass}" r="${wheelRadius}" h="${wheelWidth}"/>
@@ -100,5 +100,5 @@
 <link name="right_back">
   <inertial>
-    <origin rpy="0 0 0" xyz="-4.3520742565306136e-14 -0.022224999999999995 -2.736260904245835e-07"/>
+    <origin rpy="0 0 0" xyz="0 0 0"/>
     <mass value="${wheelMass}"/>
     <xacro:cylinder_inertia m="${wheelMass}" r="${wheelRadius}" h="${wheelWidth}"/>
@@ -125,5 +125,5 @@
 </joint>
 <joint name="right_front_rev" type="continuous">
-  <origin rpy="0 0 0" xyz="0.254 -0.254 0.101276"/>
+  <origin rpy="0 0 0" xyz="0.275 -0.3 0.14"/>
   <parent link="chassis"/>
   <child link="right_front"/>
@@ -131,5 +131,5 @@
 </joint>
 <joint name="left_front_rev" type="continuous">
-  <origin rpy="0 0 0" xyz="0.254 0.254 0.101276"/>
+  <origin rpy="0 0 0" xyz="0.275 0.23 0.14"/>
   <parent link="chassis"/>
   <child link="left_front"/>
@@ -137,5 +137,5 @@
 </joint>
 <joint name="left_back_rev" type="continuous">
-  <origin rpy="0 0 0" xyz="-0.254 0.254 0.101276"/>
+  <origin rpy="0 0 0" xyz="-0.275 0.3 0.14"/>
   <parent link="chassis"/>
   <child link="left_back"/>
@@ -143,5 +143,5 @@
 </joint>
 <joint name="right_back_rev" type="continuous">
-  <origin rpy="0 0 0" xyz="-0.254 -0.254 0.101276"/>
+  <origin rpy="0 0 0" xyz="-0.275 -0.3 0.14"/>
   <parent link="chassis"/>
   <child link="right_back"/>
@@ -150,5 +150,5 @@
 <link name="d455_back_link"/>
 <joint name="depth_cam_jnt" type="fixed">
-    <origin rpy="-2.0000019999706227e-06 0.0019999983333319994 3.139592651256459" xyz="-0.457877 0.129509 0.255037"/>
+    <origin rpy="0 0 0" xyz="0.405 -0.10 0.39"/>
   <parent link="base_link"/>
   <child link="d455_back_link"/>

Commit message: fixed more sim vis stuff

File: lunabot_sim/lunabot_description/urdf/lunabot.xacro (robot description, xacro)
@@ -45,5 +45,5 @@
   </inertial>
   <visual>
-    <origin rpy="0 0 0" xyz="-0.254 0.254 -0.101276"/>
+    <origin rpy="0 0 0" xyz="-0.275 0.3 0.14"/>
     <geometry>
       <mesh filename="package://lunabot_description/meshes/right_front.stl" scale="0.001 0.001 0.001"/>
@@ -52,5 +52,5 @@
   </visual>
   <collision>
-    <origin rpy="0 0 0" xyz="-0.254 0.254 -0.101276"/>
+    <origin rpy="0 0 0" xyz="-0.275 0.3 0.14"/>
     <geometry>
       <mesh filename="package://lunabot_description/meshes/right_front.stl" scale="0.001 0.001 0.001"/>
@@ -65,5 +65,5 @@
   </inertial>
   <visual>
-    <origin rpy="0 0 0" xyz="-0.254 -0.254 -0.101276"/>
+    <origin rpy="0 0 0" xyz="-0.275 -0.3 0.14"/>
     <geometry>
       <mesh filename="package://lunabot_description/meshes/left_front.stl" scale="0.001 0.001 0.001"/>
@@ -72,5 +72,5 @@
   </visual>
   <collision>
-    <origin rpy="0 0 0" xyz="-0.254 -0.254 -0.101276"/>
+    <origin rpy="0 0 0" xyz="-0.275 -0.3 0.14"/>
     <geometry>
       <mesh filename="package://lunabot_description/meshes/left_front.stl" scale="0.001 0.001 0.001"/>
@@ -80,10 +80,10 @@
 <link name="left_back">
   <inertial>
-    <origin rpy="0 0 0" xyz="-4.346523141407488e-14 0.02222499999999994 -2.7362609036907237e-07"/>
+    <origin rpy="0 0 0" xyz="0 0 0"/>
     <mass value="${wheelMass}"/>
     <xacro:cylinder_inertia m="${wheelMass}" r="${wheelRadius}" h="${wheelWidth}"/>
   </inertial>
   <visual>
-    <origin rpy="0 0 0" xyz="0.254 -0.254 -0.101276"/>
+    <origin rpy="0 0 0" xyz="0.275 -0.3 0.14"/>
     <geometry>
       <mesh filename="package://lunabot_description/meshes/left_back.stl" scale="0.001 0.001 0.001"/>
@@ -92,5 +92,5 @@
   </visual>
   <collision>
-    <origin rpy="0 0 0" xyz="0.254 -0.254 -0.101276"/>
+    <origin rpy="0 0 0" xyz="0.275 -0.3 0.14"/>
     <geometry>
       <mesh filename="package://lunabot_description/meshes/left_back.stl" scale="0.001 0.001 0.001"/>
@@ -105,5 +105,5 @@
   </inertial>
   <visual>
-    <origin rpy="0 0 0" xyz="0.254 0.254 -0.101276"/>
+    <origin rpy="0 0 0" xyz="0.275 0.3 0.14"/>
     <geometry>
       <mesh filename="package://lunabot_description/meshes/right_back.stl" scale="0.001 0.001 0.001"/>
@@ -112,5 +112,5 @@
   </visual>
   <collision>
-    <origin rpy="0 0 0" xyz="0.254 0.254 -0.101276"/>
+    <origin rpy="0 0 0" xyz="0.275 0.3 0.14"/>
     <geometry>
       <mesh filename="package://lunabot_description/meshes/right_back.stl" scale="0.001 0.001 0.001"/>
@@ -119,5 +119,5 @@
 </link>
 <joint name="base_link" type="fixed">
-  <origin rpy="0 0 0" xyz="0 0 -0.25"/>
+  <origin rpy="0 0 0" xyz="0 0 0"/>
   <parent link="base_link"/>
   <child link="chassis"/>
@@ -131,5 +131,5 @@
 </joint>
 <joint name="left_front_rev" type="continuous">
-  <origin rpy="0 0 0" xyz="0.275 0.23 0.14"/>
+  <origin rpy="0 0 0" xyz="0.275 0.3 0.14"/>
   <parent link="chassis"/>
   <child link="left_front"/>

Commit message: fixed camera and chassis location

File: lunabot_sim/lunabot_description/urdf/lunabot.xacro (robot description, xacro)
@@ -7,5 +7,5 @@
 <xacro:property name="chassisMass" value="55"/>
 <xacro:property name="wheelWidth" value="0.05"/>
-<xacro:property name="wheelRadius" value="0.13755"/>
+<xacro:property name="wheelRadius" value="0.15"/>
 <xacro:property name="wheelMass" value="5"/>
 <xacro:macro name="box_inertia" params="m x y z">
@@ -25,5 +25,5 @@
 <link name="chassis">
   <visual>
-    <origin rpy="0 0 0" xyz="0 0 0"/>
+    <origin rpy="0 0 0" xyz="0 0 0.215"/>
     <geometry>
       <mesh filename="package://lunabot_description/meshes/base_link.stl" scale="0.001 0.001 0.001"/>
@@ -45,5 +45,5 @@
   </inertial>
   <visual>
-    <origin rpy="0 0 0" xyz="-0.275 0.3 0.14"/>
+    <origin rpy="0 0 0" xyz="-0.275 0.3 0"/>
     <geometry>
       <mesh filename="package://lunabot_description/meshes/right_front.stl" scale="0.001 0.001 0.001"/>
@@ -52,5 +52,5 @@
   </visual>
   <collision>
-    <origin rpy="0 0 0" xyz="-0.275 0.3 0.14"/>
+    <origin rpy="0 0 0" xyz="-0.275 0.3 0"/>
     <geometry>
       <mesh filename="package://lunabot_description/meshes/right_front.stl" scale="0.001 0.001 0.001"/>
@@ -65,5 +65,5 @@
   </inertial>
   <visual>
-    <origin rpy="0 0 0" xyz="-0.275 -0.3 0.14"/>
+    <origin rpy="0 0 0" xyz="-0.275 -0.3 0"/>
     <geometry>
       <mesh filename="package://lunabot_description/meshes/left_front.stl" scale="0.001 0.001 0.001"/>
@@ -72,5 +72,5 @@
   </visual>
   <collision>
-    <origin rpy="0 0 0" xyz="-0.275 -0.3 0.14"/>
+    <origin rpy="0 0 0" xyz="-0.275 -0.3 0"/>
     <geometry>
       <mesh filename="package://lunabot_description/meshes/left_front.stl" scale="0.001 0.001 0.001"/>
@@ -85,5 +85,5 @@
   </inertial>
   <visual>
-    <origin rpy="0 0 0" xyz="0.275 -0.3 0.14"/>
+    <origin rpy="0 0 0" xyz="0.275 -0.3 0"/>
     <geometry>
       <mesh filename="package://lunabot_description/meshes/left_back.stl" scale="0.001 0.001 0.001"/>
@@ -92,5 +92,5 @@
   </visual>
   <collision>
-    <origin rpy="0 0 0" xyz="0.275 -0.3 0.14"/>
+    <origin rpy="0 0 0" xyz="0.275 -0.3 0"/>
     <geometry>
       <mesh filename="package://lunabot_description/meshes/left_back.stl" scale="0.001 0.001 0.001"/>
@@ -105,5 +105,5 @@
   </inertial>
   <visual>
-    <origin rpy="0 0 0" xyz="0.275 0.3 0.14"/>
+    <origin rpy="0 0 0" xyz="0.275 0.3 0"/>
     <geometry>
       <mesh filename="package://lunabot_description/meshes/right_back.stl" scale="0.001 0.001 0.001"/>
@@ -112,5 +112,5 @@
   </visual>
   <collision>
-    <origin rpy="0 0 0" xyz="0.275 0.3 0.14"/>
+    <origin rpy="0 0 0" xyz="0.275 0.3 0"/>
     <geometry>
       <mesh filename="package://lunabot_description/meshes/right_back.stl" scale="0.001 0.001 0.001"/>
@@ -150,5 +150,5 @@
 <link name="d455_back_link"/>
 <joint name="depth_cam_jnt" type="fixed">
-    <origin rpy="0 0 0" xyz="0.405 -0.10 0.39"/>
+    <origin rpy="0 0 0" xyz="0.405 -0.10 0.45"/>
   <parent link="base_link"/>
   <child link="d455_back_link"/>

Commit message: comp_quick_fix

File: lunabot_sim/lunabot_description/urdf/lunabot.xacro (robot description, xacro)
@@ -155,3 +155,10 @@
   <axis xyz="0.0 1.0 0.0"/>
 </joint>
+<link name="usb_cam_link"/>
+<joint name="usb_cam_jnt" type="fixed">
+    <origin rpy="0 0 3.14" xyz="-0.405 0.10 0.65"/>
+  <parent link="base_link"/>
+  <child link="usb_cam_link"/>
+  <axis xyz="0.0 1.0 0.0"/>
+</joint>
 </robot>

Commit message: chaged camera orientation

File: lunabot_sim/lunabot_description/urdf/lunabot.xacro (robot description, xacro)
@@ -157,5 +157,5 @@
 <link name="usb_cam_link"/>
 <joint name="usb_cam_jnt" type="fixed">
-    <origin rpy="0 0 3.14" xyz="-0.405 0.10 0.65"/>
+    <origin rpy="0 1.57 3.14" xyz="-0.405 0.10 0.65"/>
   <parent link="base_link"/>
   <child link="usb_cam_link"/>

Commit message: actually added transforms

File: lunabot_sim/lunabot_description/urdf/lunabot.xacro (robot description, xacro)
@@ -1,164 +1,181 @@
-<?xml version="1.0" ?>
+<?xml version="1.0"?>
 <robot name="lunabot" xmlns:xacro="http://www.ros.org/wiki/xacro">
-<xacro:property name="PI" value="3.1415926535897931"/>
-<xacro:property name="chassisHeight" value="0.2"/>
-<xacro:property name="chassisLength" value="0.82"/>
-<xacro:property name="chassisWidth" value="0.5"/>
-<xacro:property name="chassisMass" value="55"/>
-<xacro:property name="wheelWidth" value="0.05"/>
-<xacro:property name="wheelRadius" value="0.15"/>
-<xacro:property name="wheelMass" value="5"/>
-<xacro:macro name="box_inertia" params="m x y z">
-  <inertia  ixx="${m*(y*y+z*z)/12}" ixy = "0" ixz = "0"
-    iyy="${m*(x*x+z*z)/12}" iyz = "0"
-    izz="${m*(x*x+z*z)/12}"
-  />
-</xacro:macro>
-<xacro:macro name="cylinder_inertia" params="m r h">
-  <inertia  ixx="${m*(3*r*r+h*h)/12}" ixy = "0" ixz = "0"
-    iyy="${m*(3*r*r+h*h)/12}" iyz = "0"
-    izz="${m*r*r/2}"
-  />
-</xacro:macro>
-<xacro:include filename="$(find lunabot_description)/urdf/materials.xacro" />
-<link name="base_link"/>
-<link name="chassis">
-  <visual>
-    <origin rpy="0 0 0" xyz="0 0 0.215"/>
-    <geometry>
-      <mesh filename="package://lunabot_description/meshes/base_link.stl" scale="0.001 0.001 0.001"/>
-    </geometry>
-    <material name="silver"/>
-  </visual>
-  <collision>
-    <origin rpy="0 0 0" xyz="0 0 0"/>
-    <geometry>
-      <mesh filename="package://lunabot_description/meshes/base_link.stl" scale="0.001 0.001 0.001"/>
-    </geometry>
-  </collision>
-</link>
-<link name="right_front">
-  <inertial>
-    <origin rpy="0 0 0" xyz="0 0 0"/>
-    <mass value="${wheelMass}"/>
-    <xacro:cylinder_inertia m="${wheelMass}" r="${wheelRadius}" h="${wheelWidth}"/>
-  </inertial>
-  <visual>
-    <origin rpy="0 0 0" xyz="-0.275 0.3 0"/>
-    <geometry>
-      <mesh filename="package://lunabot_description/meshes/right_front.stl" scale="0.001 0.001 0.001"/>
-    </geometry>
-    <material name="silver"/>
-  </visual>
-  <collision>
-    <origin rpy="0 0 0" xyz="-0.275 0.3 0"/>
-    <geometry>
-      <mesh filename="package://lunabot_description/meshes/right_front.stl" scale="0.001 0.001 0.001"/>
-    </geometry>
-  </collision>
-</link>
-<link name="left_front">
-  <inertial>
-    <origin rpy="0 0 0" xyz="0 0 0"/>
-    <mass value="${wheelMass}"/>
-    <xacro:cylinder_inertia m="${wheelMass}" r="${wheelRadius}" h="${wheelWidth}"/>
-  </inertial>
-  <visual>
-    <origin rpy="0 0 0" xyz="-0.275 -0.3 0"/>
-    <geometry>
-      <mesh filename="package://lunabot_description/meshes/left_front.stl" scale="0.001 0.001 0.001"/>
-    </geometry>
-    <material name="silver"/>
-  </visual>
-  <collision>
-    <origin rpy="0 0 0" xyz="-0.275 -0.3 0"/>
-    <geometry>
-      <mesh filename="package://lunabot_description/meshes/left_front.stl" scale="0.001 0.001 0.001"/>
-    </geometry>
-  </collision>
-</link>
-<link name="left_back">
-  <inertial>
-    <origin rpy="0 0 0" xyz="0 0 0"/>
-    <mass value="${wheelMass}"/>
-    <xacro:cylinder_inertia m="${wheelMass}" r="${wheelRadius}" h="${wheelWidth}"/>
-  </inertial>
-  <visual>
-    <origin rpy="0 0 0" xyz="0.275 -0.3 0"/>
-    <geometry>
-      <mesh filename="package://lunabot_description/meshes/left_back.stl" scale="0.001 0.001 0.001"/>
-    </geometry>
-    <material name="silver"/>
-  </visual>
-  <collision>
-    <origin rpy="0 0 0" xyz="0.275 -0.3 0"/>
-    <geometry>
-      <mesh filename="package://lunabot_description/meshes/left_back.stl" scale="0.001 0.001 0.001"/>
-    </geometry>
-  </collision>
-</link>
-<link name="right_back">
-  <inertial>
-    <origin rpy="0 0 0" xyz="0 0 0"/>
-    <mass value="${wheelMass}"/>
-    <xacro:cylinder_inertia m="${wheelMass}" r="${wheelRadius}" h="${wheelWidth}"/>
-  </inertial>
-  <visual>
-    <origin rpy="0 0 0" xyz="0.275 0.3 0"/>
-    <geometry>
-      <mesh filename="package://lunabot_description/meshes/right_back.stl" scale="0.001 0.001 0.001"/>
-    </geometry>
-    <material name="silver"/>
-  </visual>
-  <collision>
-    <origin rpy="0 0 0" xyz="0.275 0.3 0"/>
-    <geometry>
-      <mesh filename="package://lunabot_description/meshes/right_back.stl" scale="0.001 0.001 0.001"/>
-    </geometry>
-  </collision>
-</link>
-<joint name="base_link" type="fixed">
-  <origin rpy="0 0 0" xyz="0 0 0"/>
-  <parent link="base_link"/>
-  <child link="chassis"/>
-  <axis xyz="0.0 1.0 0.0"/>
-</joint>
-<joint name="right_front_rev" type="continuous">
-  <origin rpy="0 0 0" xyz="0.275 -0.3 0.14"/>
-  <parent link="chassis"/>
-  <child link="right_front"/>
-  <axis xyz="0.0 1.0 0.0"/>
-</joint>
-<joint name="left_front_rev" type="continuous">
-  <origin rpy="0 0 0" xyz="0.275 0.3 0.14"/>
-  <parent link="chassis"/>
-  <child link="left_front"/>
-  <axis xyz="0.0 -1.0 0.0"/>
-</joint>
-<joint name="left_back_rev" type="continuous">
-  <origin rpy="0 0 0" xyz="-0.275 0.3 0.14"/>
-  <parent link="chassis"/>
-  <child link="left_back"/>
-  <axis xyz="0.0 -1.0 0.0"/>
-</joint>
-<joint name="right_back_rev" type="continuous">
-  <origin rpy="0 0 0" xyz="-0.275 -0.3 0.14"/>
-  <parent link="chassis"/>
-  <child link="right_back"/>
-  <axis xyz="0.0 1.0 0.0"/>
-</joint>
-<link name="d455_back_link"/>
-<joint name="depth_cam_jnt" type="fixed">
-    <origin rpy="0 0 0" xyz="0.405 -0.10 0.45"/>
-  <parent link="base_link"/>
-  <child link="d455_back_link"/>
-  <axis xyz="0.0 1.0 0.0"/>
-</joint>
-<link name="usb_cam_link"/>
-<joint name="usb_cam_jnt" type="fixed">
-    <origin rpy="0 1.57 3.14" xyz="-0.405 0.10 0.65"/>
-  <parent link="base_link"/>
-  <child link="usb_cam_link"/>
-  <axis xyz="0.0 1.0 0.0"/>
-</joint>
+  <xacro:property name="PI" value="3.1415926535897931" />
+  <xacro:property name="chassisHeight" value="0.2" />
+  <xacro:property name="chassisLength" value="0.82" />
+  <xacro:property name="chassisWidth" value="0.5" />
+  <xacro:property name="chassisMass" value="55" />
+  <xacro:property name="wheelWidth" value="0.05" />
+  <xacro:property name="wheelRadius" value="0.15" />
+  <xacro:property name="wheelMass" value="5" />
+  <xacro:macro name="box_inertia" params="m x y z">
+    <inertia ixx="${m*(y*y+z*z)/12}" ixy="0" ixz="0"
+      iyy="${m*(x*x+z*z)/12}" iyz="0"
+      izz="${m*(x*x+z*z)/12}"
+    />
+  </xacro:macro>
+  <xacro:macro name="cylinder_inertia" params="m r h">
+    <inertia ixx="${m*(3*r*r+h*h)/12}" ixy="0" ixz="0"
+      iyy="${m*(3*r*r+h*h)/12}" iyz="0"
+      izz="${m*r*r/2}"
+    />
+  </xacro:macro>
+  <xacro:include filename="$(find lunabot_description)/urdf/materials.xacro" />
+  <link name="base_link" />
+  <link name="chassis">
+    <visual>
+      <origin rpy="0 0 0" xyz="0 0 0.215" />
+      <geometry>
+        <mesh filename="package://lunabot_description/meshes/base_link.stl"
+          scale="0.001 0.001 0.001" />
+      </geometry>
+      <material name="silver" />
+    </visual>
+    <collision>
+      <origin rpy="0 0 0" xyz="0 0 0" />
+      <geometry>
+        <mesh filename="package://lunabot_description/meshes/base_link.stl"
+          scale="0.001 0.001 0.001" />
+      </geometry>
+    </collision>
+  </link>
+  <link name="right_front">
+    <inertial>
+      <origin rpy="0 0 0" xyz="0 0 0" />
+      <mass value="${wheelMass}" />
+      <xacro:cylinder_inertia m="${wheelMass}" r="${wheelRadius}" h="${wheelWidth}" />
+    </inertial>
+    <visual>
+      <origin rpy="0 0 0" xyz="-0.275 0.3 0" />
+      <geometry>
+        <mesh filename="package://lunabot_description/meshes/right_front.stl"
+          scale="0.001 0.001 0.001" />
+      </geometry>
+      <material name="silver" />
+    </visual>
+    <collision>
+      <origin rpy="0 0 0" xyz="-0.275 0.3 0" />
+      <geometry>
+        <mesh filename="package://lunabot_description/meshes/right_front.stl"
+          scale="0.001 0.001 0.001" />
+      </geometry>
+    </collision>
+  </link>
+  <link name="left_front">
+    <inertial>
+      <origin rpy="0 0 0" xyz="0 0 0" />
+      <mass value="${wheelMass}" />
+      <xacro:cylinder_inertia m="${wheelMass}" r="${wheelRadius}" h="${wheelWidth}" />
+    </inertial>
+    <visual>
+      <origin rpy="0 0 0" xyz="-0.275 -0.3 0" />
+      <geometry>
+        <mesh filename="package://lunabot_description/meshes/left_front.stl"
+          scale="0.001 0.001 0.001" />
+      </geometry>
+      <material name="silver" />
+    </visual>
+    <collision>
+      <origin rpy="0 0 0" xyz="-0.275 -0.3 0" />
+      <geometry>
+        <mesh filename="package://lunabot_description/meshes/left_front.stl"
+          scale="0.001 0.001 0.001" />
+      </geometry>
+    </collision>
+  </link>
+  <link name="left_back">
+    <inertial>
+      <origin rpy="0 0 0" xyz="0 0 0" />
+      <mass value="${wheelMass}" />
+      <xacro:cylinder_inertia m="${wheelMass}" r="${wheelRadius}" h="${wheelWidth}" />
+    </inertial>
+    <visual>
+      <origin rpy="0 0 0" xyz="0.275 -0.3 0" />
+      <geometry>
+        <mesh filename="package://lunabot_description/meshes/left_back.stl"
+          scale="0.001 0.001 0.001" />
+      </geometry>
+      <material name="silver" />
+    </visual>
+    <collision>
+      <origin rpy="0 0 0" xyz="0.275 -0.3 0" />
+      <geometry>
+        <mesh filename="package://lunabot_description/meshes/left_back.stl"
+          scale="0.001 0.001 0.001" />
+      </geometry>
+    </collision>
+  </link>
+  <link name="right_back">
+    <inertial>
+      <origin rpy="0 0 0" xyz="0 0 0" />
+      <mass value="${wheelMass}" />
+      <xacro:cylinder_inertia m="${wheelMass}" r="${wheelRadius}" h="${wheelWidth}" />
+    </inertial>
+    <visual>
+      <origin rpy="0 0 0" xyz="0.275 0.3 0" />
+      <geometry>
+        <mesh filename="package://lunabot_description/meshes/right_back.stl"
+          scale="0.001 0.001 0.001" />
+      </geometry>
+      <material name="silver" />
+    </visual>
+    <collision>
+      <origin rpy="0 0 0" xyz="0.275 0.3 0" />
+      <geometry>
+        <mesh filename="package://lunabot_description/meshes/right_back.stl"
+          scale="0.001 0.001 0.001" />
+      </geometry>
+    </collision>
+  </link>
+  <joint name="base_link" type="fixed">
+    <origin rpy="0 0 0" xyz="0 0 0" />
+    <parent link="base_link" />
+    <child link="chassis" />
+    <axis xyz="0.0 1.0 0.0" />
+  </joint>
+  <joint name="right_front_rev" type="continuous">
+    <origin rpy="0 0 0" xyz="0.275 -0.3 0.14" />
+    <parent link="chassis" />
+    <child link="right_front" />
+    <axis xyz="0.0 1.0 0.0" />
+  </joint>
+  <joint name="left_front_rev" type="continuous">
+    <origin rpy="0 0 0" xyz="0.275 0.3 0.14" />
+    <parent link="chassis" />
+    <child link="left_front" />
+    <axis xyz="0.0 -1.0 0.0" />
+  </joint>
+  <joint name="left_back_rev" type="continuous">
+    <origin rpy="0 0 0" xyz="-0.275 0.3 0.14" />
+    <parent link="chassis" />
+    <child link="left_back" />
+    <axis xyz="0.0 -1.0 0.0" />
+  </joint>
+  <joint name="right_back_rev" type="continuous">
+    <origin rpy="0 0 0" xyz="-0.275 -0.3 0.14" />
+    <parent link="chassis" />
+    <child link="right_back" />
+    <axis xyz="0.0 1.0 0.0" />
+  </joint>
+  <link name="d455_back_link" />
+  <joint name="depth_cam_jnt" type="fixed">
+    <origin rpy="0 0 0" xyz="0.405 -0.10 0.45" />
+    <parent link="base_link" />
+    <child link="d455_back_link" />
+    <axis xyz="0.0 1.0 0.0" />
+  </joint>
+  <link name="d455_front_link" />
+  <joint name="depth_cam_2_jnt" type="fixed">
+    <origin rpy="0 0 0" xyz="-0.508 0.25 0.5207" />
+    <parent link="base_link" />
+    <child link="d455_front_link" />
+    <axis xyz="0.0 1.0 0.0" />
+  </joint>
+  <link name="usb_cam_link" />
+  <joint name="usb_cam_jnt" type="fixed">
+    <origin rpy="0 1.57 3.14" xyz="-0.405 0.10 0.65" />
+    <parent link="base_link" />
+    <child link="usb_cam_link" />
+    <axis xyz="0.0 1.0 0.0" />
+  </joint>
 </robot>

Commit message: actually fixed the tree (for real this time)

File: lunabot_sim/lunabot_description/urdf/lunabot.xacro (robot description, xacro)
@@ -167,5 +167,5 @@
   <link name="d455_front_link" />
   <joint name="depth_cam_2_jnt" type="fixed">
-    <origin rpy="0 0 0" xyz="-0.508 0.25 0.5207" />
+    <origin rpy="3.1415926 0 0" xyz="-0.508 0.25 0.5207" />
     <parent link="base_link" />
     <child link="d455_front_link" />
