Commit message: slow down mapping to match rtabmap and some more stuff

File: lunabot_sim/lunabot_description/urdf/lunabot.xacro (robot description, xacro)
@@ -167,5 +167,5 @@
   <link name="d455_front_link" />
   <joint name="depth_cam_2_jnt" type="fixed">
-    <origin rpy="3.1415926 0 0" xyz="-0.508 0.25 0.5207" />
+    <origin rpy="0 0 3.1415926" xyz="-0.508 0.25 0.5207" />
     <parent link="base_link" />
     <child link="d455_front_link" />

Commit message: flip camera

File: lunabot_sim/lunabot_description/urdf/lunabot.xacro (robot description, xacro)
@@ -167,5 +167,5 @@
   <link name="d455_front_link" />
   <joint name="depth_cam_2_jnt" type="fixed">
-    <origin rpy="0 0 3.1415926" xyz="-0.508 0.25 0.5207" />
+    <origin rpy="3.1415926 0 3.1415926" xyz="-0.508 0.25 0.5207" />
     <parent link="base_link" />
     <child link="d455_front_link" />

Commit message: it works

File: lunabot_sim/lunabot_description/urdf/lunabot.xacro (robot description, xacro)
@@ -167,5 +167,5 @@
   <link name="d455_front_link" />
   <joint name="depth_cam_2_jnt" type="fixed">
-    <origin rpy="3.1415926 0 3.1415926" xyz="-0.508 0.25 0.5207" />
+    <origin rpy="3.1415926 0 3.1415926" xyz="-0.508 0.25 0" />
     <parent link="base_link" />
     <child link="d455_front_link" />

Commit message: Tuning values

File: lunabot_sim/lunabot_description/urdf/lunabot.xacro (robot description, xacro)
@@ -167,5 +167,5 @@
   <link name="d455_front_link" />
   <joint name="depth_cam_2_jnt" type="fixed">
-    <origin rpy="3.1415926 0 3.1415926" xyz="-0.508 0.25 0" />
+    <origin rpy="3.1415926 0 3.1415926" xyz="-0.508 0.25 0.5207" />
     <parent link="base_link" />
     <child link="d455_front_link" />

Commit message: make camera actually at right height, and costmap find new pointclouds

File: lunabot_sim/lunabot_description/urdf/lunabot.xacro (robot description, xacro)
@@ -167,5 +167,5 @@
   <link name="d455_front_link" />
   <joint name="depth_cam_2_jnt" type="fixed">
-    <origin rpy="3.1415926 0 3.1415926" xyz="-0.508 0.25 0.5207" />
+    <origin rpy="3.1415926 0 3.1415926" xyz="-0.508 0.508 0.5207" />
     <parent link="base_link" />
     <child link="d455_front_link" />

Commit message: multicam works but at 3hz

File: lunabot_sim/lunabot_description/urdf/lunabot.xacro (robot description, xacro)
@@ -167,5 +167,5 @@
   <link name="d455_front_link" />
   <joint name="depth_cam_2_jnt" type="fixed">
-    <origin rpy="3.1415926 0 3.1415926" xyz="-0.508 0.508 0.5207" />
+    <origin rpy="3.1415926 0 3.1415926" xyz="-0.334 0 0.508" />
     <parent link="base_link" />
     <child link="d455_front_link" />

Commit message: fixed transforms

File: lunabot_sim/lunabot_description/urdf/lunabot.xacro (robot description, xacro)
@@ -167,5 +167,5 @@
   <link name="d455_front_link" />
   <joint name="depth_cam_2_jnt" type="fixed">
-    <origin rpy="3.1415926 0 3.1415926" xyz="-0.508 0.25 0" />
+    <origin rpy="3.1415926 0 3.1415926" xyz="-.484 0 0.508" />
     <parent link="base_link" />
     <child link="d455_front_link" />

Commit message: change transforms for testing

File: lunabot_sim/lunabot_description/urdf/lunabot.xacro (robot description, xacro)
@@ -160,5 +160,5 @@
   <link name="d455_back_link" />
   <joint name="depth_cam_jnt" type="fixed">
-    <origin rpy="0 0 0" xyz="0.405 -0.10 0.45" />
+    <origin rpy="0 0 0" xyz="0 0 0" />
     <parent link="base_link" />
     <child link="d455_back_link" />
@@ -167,5 +167,5 @@
   <link name="d455_front_link" />
   <joint name="depth_cam_2_jnt" type="fixed">
-    <origin rpy="3.1415926 0 3.1415926" xyz="-.484 0 0.508" />
+    <origin rpy="0 0 3.1415926" xyz="-.2032 0 0" />
     <parent link="base_link" />
     <child link="d455_front_link" />

Commit message: Three Cameras??

File: lunabot_sim/lunabot_description/urdf/lunabot.xacro (robot description, xacro)
@@ -172,4 +172,11 @@
     <axis xyz="0.0 1.0 0.0" />
   </joint>
+  <link name="d435_extra_link" />
+  <joint name="depth_cam_3_jnt" type="fixed">
+    <origin rpy="0 0 1.57079632679489661" xyz="-.1016 0 0" />
+    <parent link="base_link" />
+    <child link="d435_extra_link" />
+    <axis xyz="0.0 1.0 0.0" />
+  </joint>
   <link name="usb_cam_link" />
   <joint name="usb_cam_jnt" type="fixed">

Commit message: fourth camera?!??!!

File: lunabot_sim/lunabot_description/urdf/lunabot.xacro (robot description, xacro)
@@ -172,9 +172,16 @@
     <axis xyz="0.0 1.0 0.0" />
   </joint>
-  <link name="d435_extra_link" />
+  <link name="d435_right_link" />
   <joint name="depth_cam_3_jnt" type="fixed">
     <origin rpy="0 0 1.57079632679489661" xyz="-.1016 0 0" />
     <parent link="base_link" />
-    <child link="d435_extra_link" />
+    <child link="d435_right_link" />
+    <axis xyz="0.0 1.0 0.0" />
+  </joint>
+  <link name="d435_left_link" />
+  <joint name="depth_cam_4_jnt" type="fixed">
+    <origin rpy="0 0 14.7123889803846" xyz="-.1016 0 0" />
+    <parent link="base_link" />
+    <child link="d435_left_link" />
     <axis xyz="0.0 1.0 0.0" />
   </joint>

Commit message: fix positions of cameras

File: lunabot_sim/lunabot_description/urdf/lunabot.xacro (robot description, xacro)
@@ -181,5 +181,5 @@
   <link name="d435_left_link" />
   <joint name="depth_cam_4_jnt" type="fixed">
-    <origin rpy="0 0 14.7123889803846" xyz="-.1016 0 0" />
+    <origin rpy="0 0 4.7123889803846" xyz="-.1016 0 0" />
     <parent link="base_link" />
     <child link="d435_left_link" />

Commit message: new transforms

File: lunabot_sim/lunabot_description/urdf/lunabot.xacro (robot description, xacro)
@@ -159,6 +159,6 @@
   </joint>
   <link name="d455_back_link" />
-  <joint name="depth_cam_jnt" type="fixed">
-    <origin rpy="0 0 0" xyz="0 0 0" />
+  <joint name="depth_cam_back_jnt" type="fixed">
+    <origin rpy="3.14159265359 0 3.14159265359" xyz="-0.3302 0 0.508" />
     <parent link="base_link" />
     <child link="d455_back_link" />
@@ -166,6 +166,6 @@
   </joint>
   <link name="d455_front_link" />
-  <joint name="depth_cam_2_jnt" type="fixed">
-    <origin rpy="0 0 3.1415926" xyz="-.2032 0 0" />
+  <joint name="depth_cam_front_jnt" type="fixed">
+    <origin rpy="0 0 0" xyz="0.5842 -0.2032 0.381" />
     <parent link="base_link" />
     <child link="d455_front_link" />

Commit message: change transforms for test bot

File: lunabot_sim/lunabot_description/urdf/lunabot.xacro (robot description, xacro)
@@ -148,11 +148,17 @@
   <axis xyz="0.0 1.0 0.0"/>
 </joint>
-<link name="d455_back_link"/>
-<joint name="depth_cam_jnt" type="fixed">
-    <origin rpy="0 0 0" xyz="0.405 -0.10 0.45"/>
-  <parent link="base_link"/>
-  <child link="d455_back_link"/>
-  <axis xyz="0.0 1.0 0.0"/>
-</joint>
+  <joint name="depth_cam_back_jnt" type="fixed">
+    <origin rpy="3.14159265359 0 3.14159265359" xyz="-0.3302 0 0.508" />
+    <parent link="base_link" />
+    <child link="d455_back_link" />
+    <axis xyz="0.0 1.0 0.0" />
+  </joint>
+  <link name="d455_front_link" />
+  <joint name="depth_cam_front_jnt" type="fixed">
+    <origin rpy="0 0 0" xyz="0.5842 -0.2032 0.381" />
+    <parent link="base_link" />
+    <child link="d455_front_link" />
+    <axis xyz="0.0 1.0 0.0" />
+  </joint>
 <link name="usb_cam_link"/>
 <joint name="usb_cam_jnt" type="fixed">

Commit message: fix typo

File: lunabot_sim/lunabot_description/urdf/lunabot.xacro (robot description, xacro)
@@ -148,17 +148,18 @@
   <axis xyz="0.0 1.0 0.0"/>
 </joint>
-  <joint name="depth_cam_back_jnt" type="fixed">
-    <origin rpy="3.14159265359 0 3.14159265359" xyz="-0.3302 0 0.508" />
-    <parent link="base_link" />
-    <child link="d455_back_link" />
-    <axis xyz="0.0 1.0 0.0" />
-  </joint>
-  <link name="d455_front_link" />
-  <joint name="depth_cam_front_jnt" type="fixed">
-    <origin rpy="0 0 0" xyz="0.5842 -0.2032 0.381" />
-    <parent link="base_link" />
-    <child link="d455_front_link" />
-    <axis xyz="0.0 1.0 0.0" />
-  </joint>
+<link name="d455_back_link"
+<joint name="depth_cam_back_jnt" type="fixed">
+  <origin rpy="3.14159265359 0 3.14159265359" xyz="-0.3302 0 0.508" />
+  <parent link="base_link" />
+  <child link="d455_back_link" />
+  <axis xyz="0.0 1.0 0.0" />
+</joint>
+<link name="d455_front_link" />
+<joint name="depth_cam_front_jnt" type="fixed">
+  <origin rpy="0 0 0" xyz="0.5842 -0.2032 0.381" />
+  <parent link="base_link" />
+  <child link="d455_front_link" />
+  <axis xyz="0.0 1.0 0.0" />
+</joint>
 <link name="usb_cam_link"/>
 <joint name="usb_cam_jnt" type="fixed">

Commit message: fix typo

File: lunabot_sim/lunabot_description/urdf/lunabot.xacro (robot description, xacro)
@@ -148,5 +148,5 @@
   <axis xyz="0.0 1.0 0.0"/>
 </joint>
-<link name="d455_back_link"
+<link name="d455_back_link" />
 <joint name="depth_cam_back_jnt" type="fixed">
   <origin rpy="3.14159265359 0 3.14159265359" xyz="-0.3302 0 0.508" />

Commit message: updated transforms

File: lunabot_sim/lunabot_description/urdf/lunabot.xacro (robot description, xacro)
@@ -160,5 +160,5 @@
   <link name="d455_back_link" />
   <joint name="depth_cam_back_jnt" type="fixed">
-    <origin rpy="3.14159265359 0 3.14159265359" xyz="-0.3302 0 0.508" />
+    <origin rpy="0 0 3.14159265359" xyz="-0.3302 0 0.5715" />
     <parent link="base_link" />
     <child link="d455_back_link" />
@@ -167,5 +167,5 @@
   <link name="d455_front_link" />
   <joint name="depth_cam_front_jnt" type="fixed">
-    <origin rpy="0 0 0" xyz="0.5842 -0.2032 0.381" />
+    <origin rpy="0 0 0" xyz="0.5842 -0.2032 0.356" />
     <parent link="base_link" />
     <child link="d455_front_link" />

Commit message: allow for different angles on front cam
change pitch on jnt2

File: lunabot_sim/lunabot_description/urdf/lunabot.xacro (robot description, xacro)
@@ -166,7 +166,13 @@
   </joint>
   <link name="d455_front_link" />
+  <joint name="depth_cam_front_jnt2" type="fixed">
+    <origin rpy="0 0 0" xyz="0.5207 -0.2032 0.356" />
+    <parent link="base_link" />
+    <child link="depth_cam_front_jnt" />
+    <axis xyz="0.0 1.0 0.0" />
+  </joint>
   <joint name="depth_cam_front_jnt" type="fixed">
-    <origin rpy="0 0 0" xyz="0.5842 -0.2032 0.356" />
-    <parent link="base_link" />
+    <origin rpy="0 0 0" xyz="0.0635 0 0" />
+    <parent link="depth_cam_front_jnt2" />
     <child link="d455_front_link" />
     <axis xyz="0.0 1.0 0.0" />

Commit message: Update lunabot.xacro

File: lunabot_sim/lunabot_description/urdf/lunabot.xacro (robot description, xacro)
@@ -166,13 +166,14 @@
   </joint>
   <link name="d455_front_link" />
-  <joint name="depth_cam_front_jnt2" type="fixed">
-    <origin rpy="0 0 0" xyz="0.5207 -0.2032 0.356" />
-    <parent link="base_link" />
-    <child link="depth_cam_front_jnt" />
+  <link name="d455_front_axis_link" />
+  <joint name="depth_cam_front_axis_jnt" type="fixed">
+    <origin rpy="0 0.5 0" xyz="0.5207 -0.2032 0.356" />
+    <parent link="base_link" />
+    <child link="d455_front_axis_link" />
     <axis xyz="0.0 1.0 0.0" />
   </joint>
   <joint name="depth_cam_front_jnt" type="fixed">
     <origin rpy="0 0 0" xyz="0.0635 0 0" />
-    <parent link="depth_cam_front_jnt2" />
+    <parent link="d455_front_axis_link" />
     <child link="d455_front_link" />
     <axis xyz="0.0 1.0 0.0" />

Commit message: adjust frame for tilted camera

File: lunabot_sim/lunabot_description/urdf/lunabot.xacro (robot description, xacro)
@@ -166,7 +166,14 @@
   </joint>
   <link name="d455_front_link" />
+  <link name="d455_front_axis_link" />
+  <joint name="depth_cam_front_axis_jnt" type="fixed">
+    <origin rpy="0 0.401 0" xyz="0.5207 -0.2032 0.356" />
+    <parent link="base_link" />
+    <child link="d455_front_axis_link" />
+    <axis xyz="0.0 1.0 0.0" />
+  </joint>
   <joint name="depth_cam_front_jnt" type="fixed">
-    <origin rpy="0 0 0" xyz="0.5842 -0.2032 0.356" />
-    <parent link="base_link" />
+    <origin rpy="0 0 0" xyz="0.0635 0.0 0.0" />
+    <parent link="d455_front_axis_link" />
     <child link="d455_front_link" />
     <axis xyz="0.0 1.0 0.0" />

Commit message: switch back and right cameras

File: lunabot_sim/lunabot_description/urdf/lunabot.xacro (robot description, xacro)
@@ -160,5 +160,5 @@
   <link name="d455_back_link" />
   <joint name="depth_cam_back_jnt" type="fixed">
-    <origin rpy="0 0 3.14159265359" xyz="-0.3302 0 0.5715" />
+    <origin rpy="3.14159265359 0 3.14159265359" xyz="-0.3302 0 0.5715" />
     <parent link="base_link" />
     <child link="d455_back_link" />
