Commit message: roboto existo! turns out gazebo doesn't like our STLs, might be an encoding issue

File: lunabot_description/urdf/dummy_bot.xacro (robot description, xacro)
@@ -21,4 +21,5 @@
   />
 </xacro:macro>
+<!-- NOTE: STL files don't work in gazebo with binary encoding, try ASCII instead -->
 <xacro:include filename="$(find lunabot_description)/urdf/materials.xacro" />
 <xacro:include filename="$(find lunabot_description)/urdf/dummy_bot.trans" />
@@ -33,5 +34,6 @@
     <origin rpy="0 0 0" xyz="0 0 0"/>
     <geometry>
-      <mesh filename="package://lunabot_description/meshes/base_link.stl" scale="0.001 0.001 0.001"/>
+      <!-- <mesh filename="package://lunabot_description/meshes/base_link.stl" scale="0.001 0.001 0.001"/> -->
+       <box size="0.9 0.5 0.1"/>
     </geometry>
     <material name="silver"/>
@@ -40,5 +42,6 @@
     <origin rpy="0 0 0" xyz="0 0 0"/>
     <geometry>
-      <mesh filename="package://lunabot_description/meshes/base_link.stl" scale="0.001 0.001 0.001"/>
+      <!-- <mesh filename="package://lunabot_description/meshes/base_link.stl" scale="0.001 0.001 0.001"/> -->
+      <box size="0.5 0.5 0.1"/>
     </geometry>
   </collision>
@@ -51,14 +54,20 @@
   </inertial>
   <visual>
-    <origin rpy="0 0 0" xyz="-0.254 0.254 -0.101276"/>
+    <!-- <origin rpy="0 0 0" xyz="-0.254 0.254 -0.101276"/> -->
+    <!-- <origin rpy="1.57079633 0 0" xyz="0.175 -0.3125 0"/> -->
+    <origin rpy="1.57079633 0 0" xyz="0 0 0"/>
     <geometry>
-      <mesh filename="package://lunabot_description/meshes/right_front.stl" scale="0.001 0.001 0.001"/>
+      <!-- <mesh filename="package://lunabot_description/meshes/right_front.stl" scale="0.001 0.001 0.001"/> -->
+      <cylinder radius="0.2" length="0.125" />
     </geometry>
     <material name="silver"/>
   </visual>
   <collision>
-    <origin rpy="0 0 0" xyz="-0.254 0.254 -0.101276"/>
+    <!-- <origin rpy="0 0 0" xyz="-0.254 0.254 -0.101276"/> -->
+    <!-- <origin rpy="1.57079633 0 0" xyz="0.175 -0.3125 0"/> -->
+    <origin rpy="1.57079633 0 0" xyz="0 0 0"/>
     <geometry>
-      <mesh filename="package://lunabot_description/meshes/right_front.stl" scale="0.001 0.001 0.001"/>
+      <!-- <mesh filename="package://lunabot_description/meshes/right_front.stl" scale="0.001 0.001 0.001"/> -->
+      <cylinder radius="0.2" length="0.125" />
     </geometry>
   </collision>
@@ -71,14 +80,18 @@
   </inertial>
   <visual>
-    <origin rpy="0 0 0" xyz="-0.254 -0.254 -0.101276"/>
+    <!-- <origin rpy="0 0 0" xyz="-0.254 -0.254 -0.101276"/> -->
+    <origin rpy="1.57079633 0 0" xyz="0 0 0"/>
     <geometry>
-      <mesh filename="package://lunabot_description/meshes/left_front.stl" scale="0.001 0.001 0.001"/>
+      <!-- <mesh filename="package://lunabot_description/meshes/left_front.stl" scale="0.001 0.001 0.001"/> -->
+      <cylinder radius="0.2" length="0.125" />
     </geometry>
     <material name="silver"/>
   </visual>
   <collision>
-    <origin rpy="0 0 0" xyz="-0.254 -0.254 -0.101276"/>
+    <!-- <origin rpy="0 0 0" xyz="-0.254 -0.254 -0.101276"/> -->
+    <origin rpy="1.57079633 0 0" xyz="0 0 0"/>
     <geometry>
-      <mesh filename="package://lunabot_description/meshes/left_front.stl" scale="0.001 0.001 0.001"/>
+      <!-- <mesh filename="package://lunabot_description/meshes/left_front.stl" scale="0.001 0.001 0.001"/> -->
+      <cylinder radius="0.2" length="0.125" />
     </geometry>
   </collision>
@@ -91,14 +104,18 @@
   </inertial>
   <visual>
-    <origin rpy="0 0 0" xyz="0.254 -0.254 -0.101276"/>
+    <!-- <origin rpy="0 0 0" xyz="0.254 -0.254 -0.101276"/> -->
+    <origin rpy="1.57079633 0 0" xyz="0 0 0"/>
     <geometry>
-      <mesh filename="package://lunabot_description/meshes/left_back.stl" scale="0.001 0.001 0.001"/>
+      <!-- <mesh filename="package://lunabot_description/meshes/left_back.stl" scale="0.001 0.001 0.001"/> -->
+      <cylinder radius="0.2" length="0.125" />
     </geometry>
     <material name="silver"/>
   </visual>
   <collision>
-    <origin rpy="0 0 0" xyz="0.254 -0.254 -0.101276"/>
+    <!-- <origin rpy="0 0 0" xyz="0.254 -0.254 -0.101276"/> -->
+    <origin rpy="1.57079633 0 0" xyz="0 0 0"/>
     <geometry>
-      <mesh filename="package://lunabot_description/meshes/left_back.stl" scale="0.001 0.001 0.001"/>
+      <!-- <mesh filename="package://lunabot_description/meshes/left_back.stl" scale="0.001 0.001 0.001"/> -->
+      <cylinder radius="0.2" length="0.125" />
     </geometry>
   </collision>
@@ -111,19 +128,25 @@
   </inertial>
   <visual>
-    <origin rpy="0 0 0" xyz="0.254 0.254 -0.101276"/>
+    <!-- <origin rpy="0 0 0" xyz="0.254 0.254 -0.101276"/> -->
+    <origin rpy="1.57079633 0 0" xyz="0 0 0"/>
     <geometry>
-      <mesh filename="package://lunabot_description/meshes/right_back.stl" scale="0.001 0.001 0.001"/>
+      <!-- <mesh filename="package://lunabot_description/meshes/right_back.stl" scale="0.001 0.001 0.001"/> -->
+      <cylinder radius="0.2" length="0.125" />
     </geometry>
     <material name="silver"/>
   </visual>
   <collision>
-    <origin rpy="0 0 0" xyz="0.254 0.254 -0.101276"/>
+    <!-- <origin rpy="0 0 0" xyz="0.254 0.254 -0.101276"/> -->
+    <origin rpy="1.57079633 0 0" xyz="0 0 0"/>
     <geometry>
-      <mesh filename="package://lunabot_description/meshes/right_back.stl" scale="0.001 0.001 0.001"/>
+      <!-- <mesh filename="package://lunabot_description/meshes/right_back.stl" scale="0.001 0.001 0.001"/> -->
+      <cylinder radius="0.2" length="0.125" />
     </geometry>
   </collision>
 </link>
+<!-- rpy="1.57079633 0 0" xyz="0.175 -0.3125 0" -->
 <joint name="right_front_rev" type="continuous">
-  <origin rpy="0 0 0" xyz="0.254 -0.254 0.101276"/>
+  <!-- <origin rpy="0 0 0" xyz="0.254 -0.254 0.101276"/> -->
+  <origin rpy="0 0 0" xyz="0.25 -0.3125 0"/>
   <parent link="base_link"/>
   <child link="right_front"/>
@@ -131,5 +154,6 @@
 </joint>
 <joint name="left_front_rev" type="continuous">
-  <origin rpy="0 0 0" xyz="0.254 0.254 0.101276"/>
+  <!-- <origin rpy="0 0 0" xyz="0.254 0.254 0.101276"/> -->
+  <origin rpy="0 0 0" xyz="0.25 0.3125 0"/>
   <parent link="base_link"/>
   <child link="left_front"/>
@@ -137,5 +161,6 @@
 </joint>
 <joint name="left_back_rev" type="continuous">
-  <origin rpy="0 0 0" xyz="-0.254 0.254 0.101276"/>
+  <!-- <origin rpy="0 0 0" xyz="-0.254 0.254 0.101276"/> -->
+  <origin rpy="0 0 0" xyz="-0.25 0.3125 0"/>
   <parent link="base_link"/>
   <child link="left_back"/>
@@ -143,5 +168,6 @@
 </joint>
 <joint name="right_back_rev" type="continuous">
-  <origin rpy="0 0 0" xyz="-0.254 -0.254 0.101276"/>
+  <!-- <origin rpy="0 0 0" xyz="-0.254 -0.254 0.101276"/> -->
+  <origin rpy="0 0 0" xyz="-0.25 -0.3125 0"/>
   <parent link="base_link"/>
   <child link="right_back"/>

Commit message: backing up gazebo stuff

File: lunabot_description/urdf/dummy_bot.xacro (robot description, xacro)
@@ -3,8 +3,8 @@
 <xacro:property name="PI" value="3.1415926535897931"/>
 <xacro:property name="chassisHeight" value="0.1"/>
-<xacro:property name="chassisLength" value="0.8"/>
+<xacro:property name="chassisLength" value="0.9"/>
 <xacro:property name="chassisWidth" value="0.5"/>
 <xacro:property name="chassisMass" value="50"/>
-<xacro:property name="wheelWidth" value="0.05"/>
+<xacro:property name="wheelWidth" value="0.125"/>
 <xacro:property name="wheelRadius" value="0.2"/>
 <xacro:property name="wheelMass" value="5"/>
@@ -23,9 +23,9 @@
 <!-- NOTE: STL files don't work in gazebo with binary encoding, try ASCII instead -->
 <xacro:include filename="$(find lunabot_description)/urdf/materials.xacro" />
-<xacro:include filename="$(find lunabot_description)/urdf/dummy_bot.trans" />
-<xacro:include filename="$(find lunabot_description)/urdf/dummy_bot.gazebo" />
+<!-- <xacro:include filename="$(find lunabot_description)/urdf/dummy_bot.trans" /> -->
+<!-- <xacro:include filename="$(find lunabot_description)/urdf/dummy_bot.gazebo" /> -->
 <link name="base_link">
   <inertial>
-    <origin rpy="0 0 0" xyz="0 0.0 0.08835894305363262"/>
+    <origin rpy="0 0 0" xyz="0 0 0"/>
     <mass value="${chassisMass}"/>
     <xacro:box_inertia m="${chassisMass}" x="${chassisLength}" y="${chassisWidth}" z="${chassisHeight}"/>
@@ -35,5 +35,5 @@
     <geometry>
       <!-- <mesh filename="package://lunabot_description/meshes/base_link.stl" scale="0.001 0.001 0.001"/> -->
-       <box size="0.9 0.5 0.1"/>
+      <box size="${chassisLength} ${chassisWidth} ${chassisHeight}"/>
     </geometry>
     <material name="silver"/>
@@ -43,135 +43,39 @@
     <geometry>
       <!-- <mesh filename="package://lunabot_description/meshes/base_link.stl" scale="0.001 0.001 0.001"/> -->
-      <box size="0.5 0.5 0.1"/>
+      <box size="${chassisLength} ${chassisWidth} ${chassisHeight}"/>
     </geometry>
   </collision>
 </link>
-<link name="right_front">
-  <inertial>
-    <origin rpy="0 0 0" xyz="-4.3576253716537394e-14 -0.022224999999999995 -2.736260904245835e-07"/>
-    <mass value="${wheelMass}"/>
-    <xacro:cylinder_inertia m="${wheelMass}" r="${wheelRadius}" h="${wheelWidth}"/>
-  </inertial>
-  <visual>
-    <!-- <origin rpy="0 0 0" xyz="-0.254 0.254 -0.101276"/> -->
-    <!-- <origin rpy="1.57079633 0 0" xyz="0.175 -0.3125 0"/> -->
-    <origin rpy="1.57079633 0 0" xyz="0 0 0"/>
-    <geometry>
-      <!-- <mesh filename="package://lunabot_description/meshes/right_front.stl" scale="0.001 0.001 0.001"/> -->
-      <cylinder radius="0.2" length="0.125" />
-    </geometry>
-    <material name="silver"/>
-  </visual>
-  <collision>
-    <!-- <origin rpy="0 0 0" xyz="-0.254 0.254 -0.101276"/> -->
-    <!-- <origin rpy="1.57079633 0 0" xyz="0.175 -0.3125 0"/> -->
-    <origin rpy="1.57079633 0 0" xyz="0 0 0"/>
-    <geometry>
-      <!-- <mesh filename="package://lunabot_description/meshes/right_front.stl" scale="0.001 0.001 0.001"/> -->
-      <cylinder radius="0.2" length="0.125" />
-    </geometry>
-  </collision>
-</link>
-<link name="left_front">
-  <inertial>
-    <origin rpy="0 0 0" xyz="-4.3576253716537394e-14 0.02222499999999994 -2.736260904245835e-07"/>
-    <mass value="${wheelMass}"/>
-    <xacro:cylinder_inertia m="${wheelMass}" r="${wheelRadius}" h="${wheelWidth}"/>
-  </inertial>
-  <visual>
-    <!-- <origin rpy="0 0 0" xyz="-0.254 -0.254 -0.101276"/> -->
-    <origin rpy="1.57079633 0 0" xyz="0 0 0"/>
-    <geometry>
-      <!-- <mesh filename="package://lunabot_description/meshes/left_front.stl" scale="0.001 0.001 0.001"/> -->
-      <cylinder radius="0.2" length="0.125" />
-    </geometry>
-    <material name="silver"/>
-  </visual>
-  <collision>
-    <!-- <origin rpy="0 0 0" xyz="-0.254 -0.254 -0.101276"/> -->
-    <origin rpy="1.57079633 0 0" xyz="0 0 0"/>
-    <geometry>
-      <!-- <mesh filename="package://lunabot_description/meshes/left_front.stl" scale="0.001 0.001 0.001"/> -->
-      <cylinder radius="0.2" length="0.125" />
-    </geometry>
-  </collision>
-</link>
-<link name="left_back">
-  <inertial>
-    <origin rpy="0 0 0" xyz="-4.346523141407488e-14 0.02222499999999994 -2.7362609036907237e-07"/>
-    <mass value="${wheelMass}"/>
-    <xacro:cylinder_inertia m="${wheelMass}" r="${wheelRadius}" h="${wheelWidth}"/>
-  </inertial>
-  <visual>
-    <!-- <origin rpy="0 0 0" xyz="0.254 -0.254 -0.101276"/> -->
-    <origin rpy="1.57079633 0 0" xyz="0 0 0"/>
-    <geometry>
-      <!-- <mesh filename="package://lunabot_description/meshes/left_back.stl" scale="0.001 0.001 0.001"/> -->
-      <cylinder radius="0.2" length="0.125" />
-    </geometry>
-    <material name="silver"/>
-  </visual>
-  <collision>
-    <!-- <origin rpy="0 0 0" xyz="0.254 -0.254 -0.101276"/> -->
-    <origin rpy="1.57079633 0 0" xyz="0 0 0"/>
-    <geometry>
-      <!-- <mesh filename="package://lunabot_description/meshes/left_back.stl" scale="0.001 0.001 0.001"/> -->
-      <cylinder radius="0.2" length="0.125" />
-    </geometry>
-  </collision>
-</link>
-<link name="right_back">
-  <inertial>
-    <origin rpy="0 0 0" xyz="-4.3520742565306136e-14 -0.022224999999999995 -2.736260904245835e-07"/>
-    <mass value="${wheelMass}"/>
-    <xacro:cylinder_inertia m="${wheelMass}" r="${wheelRadius}" h="${wheelWidth}"/>
-  </inertial>
-  <visual>
-    <!-- <origin rpy="0 0 0" xyz="0.254 0.254 -0.101276"/> -->
-    <origin rpy="1.57079633 0 0" xyz="0 0 0"/>
-    <geometry>
-      <!-- <mesh filename="package://lunabot_description/meshes/right_back.stl" scale="0.001 0.001 0.001"/> -->
-      <cylinder radius="0.2" length="0.125" />
-    </geometry>
-    <material name="silver"/>
-  </visual>
-  <collision>
-    <!-- <origin rpy="0 0 0" xyz="0.254 0.254 -0.101276"/> -->
-    <origin rpy="1.57079633 0 0" xyz="0 0 0"/>
-    <geometry>
-      <!-- <mesh filename="package://lunabot_description/meshes/right_back.stl" scale="0.001 0.001 0.001"/> -->
-      <cylinder radius="0.2" length="0.125" />
-    </geometry>
-  </collision>
-</link>
-<!-- rpy="1.57079633 0 0" xyz="0.175 -0.3125 0" -->
-<joint name="right_front_rev" type="continuous">
-  <!-- <origin rpy="0 0 0" xyz="0.254 -0.254 0.101276"/> -->
-  <origin rpy="0 0 0" xyz="0.25 -0.3125 0"/>
-  <parent link="base_link"/>
-  <child link="right_front"/>
-  <axis xyz="0.0 1.0 0.0"/>
-</joint>
-<joint name="left_front_rev" type="continuous">
-  <!-- <origin rpy="0 0 0" xyz="0.254 0.254 0.101276"/> -->
-  <origin rpy="0 0 0" xyz="0.25 0.3125 0"/>
-  <parent link="base_link"/>
-  <child link="left_front"/>
-  <axis xyz="0.0 -1.0 0.0"/>
-</joint>
-<joint name="left_back_rev" type="continuous">
-  <!-- <origin rpy="0 0 0" xyz="-0.254 0.254 0.101276"/> -->
-  <origin rpy="0 0 0" xyz="-0.25 0.3125 0"/>
-  <parent link="base_link"/>
-  <child link="left_back"/>
-  <axis xyz="0.0 -1.0 0.0"/>
-</joint>
-<joint name="right_back_rev" type="continuous">
-  <!-- <origin rpy="0 0 0" xyz="-0.254 -0.254 0.101276"/> -->
-  <origin rpy="0 0 0" xyz="-0.25 -0.3125 0"/>
-  <parent link="base_link"/>
-  <child link="right_back"/>
-  <axis xyz="0.0 1.0 0.0"/>
-</joint>
+<!-- wheel macro -->
+<xacro:macro name="wheel" params="name x y">
+  <link name="${name}">
+    <inertial>
+      <origin xyz="0 0 0"/>
+      <mass value="${wheelMass}"/>
+      <xacro:cylinder_inertia m="${wheelMass}" r="${wheelRadius}" h="${wheelWidth}"/>
+    </inertial>
+    <visual>
+      <origin rpy="1.5708 0 0" xyz="0 0 0"/>
+      <geometry><cylinder radius="${wheelRadius}" length="${wheelWidth}"/></geometry>
+      <material name="silver"/>
+    </visual>
+    <collision>
+      <origin rpy="1.5708 0 0" xyz="0 0 0"/>
+      <geometry><cylinder radius="${wheelRadius}" length="${wheelWidth}"/></geometry>
+    </collision>
+  </link>
+  <joint name="${name}_rev" type="continuous">
+    <origin rpy="0 0 0" xyz="${x} ${y} 0"/>
+    <parent link="base_link"/>
+    <child link="${name}"/>
+    <axis xyz="0 1 0"/>
+    <limit effort="10.0" velocity="100.0"/>
+  </joint>
+</xacro:macro>
+<!-- Instantiate wheels -->
+<xacro:wheel name="left_front"  x="0.25" y="0.32"/>
+<xacro:wheel name="left_back"   x="-0.25" y="0.32"/>
+<xacro:wheel name="right_front" x="0.25" y="-0.32"/>
+<xacro:wheel name="right_back"  x="-0.25" y="-0.32"/>
 <!-- <xacro:include filename="package://mining_arena_gazebo/realsense_ros_gazebo/xacro/depthcam.xacro"/> -->
 <!-- <xacro:realsense_d435 sensor_name="d435_forward" parent_link="base_link" rate="10"> -->
@@ -181,3 +85,87 @@
   <!-- <origin xyz="0.000 0.20 0.482" rpy="0 0 3.1415" /> -->
 <!-- </xacro:realsense_d435> -->
+<ros2_control name="GazeboSystem" type="system">
+  <hardware>
+    <plugin>gazebo_ros2_control/GazeboSystem</plugin>
+  </hardware>
+  <joint name="right_front_rev">
+    <command_interface name="velocity"/>
+    <state_interface name="position"/>
+    <state_interface name="velocity"/>
+    <state_interface name="effort"/>
+  </joint>
+  <joint name="left_front_rev">
+    <command_interface name="velocity"/>
+    <state_interface name="position"/>
+    <state_interface name="velocity"/>
+    <state_interface name="effort"/>
+  </joint>
+  <joint name="right_back_rev">
+    <command_interface name="velocity"/>
+    <state_interface name="position"/>
+    <state_interface name="velocity"/>
+    <state_interface name="effort"/>
+  </joint>
+  <joint name="left_back_rev">
+    <command_interface name="velocity"/>
+    <state_interface name="position"/>
+    <state_interface name="velocity"/>
+    <state_interface name="effort"/>
+  </joint>
+</ros2_control>
+<!-- Transmissions -->
+<xacro:macro name="transmission" params="joint_name">
+  <transmission name="${joint_name}_trans">
+    <type>transmission_interface/SimpleTransmission</type>
+    <joint name="${joint_name}">
+      <hardwareInterface>hardware_interface/VelocityJointInterface</hardwareInterface>
+    </joint>
+    <actuator name="${joint_name}_motor">
+      <hardwareInterface>hardware_interface/VelocityJointInterface</hardwareInterface>
+      <mechanicalReduction>1.0</mechanicalReduction>
+    </actuator>
+  </transmission>
+</xacro:macro>
+<xacro:transmission joint_name="left_front_rev"/>
+<xacro:transmission joint_name="left_back_rev"/>
+<xacro:transmission joint_name="right_front_rev"/>
+<xacro:transmission joint_name="right_back_rev"/>
+<!-- diff drive controller in gazebo -->
+<gazebo reference="base_link">
+  <plugin name="diff_drive_controller" filename="libgazebo_ros_diff_drive.so">
+    <updateRate>60</updateRate>
+    <leftJoint>left_front_rev left_back_rev</leftJoint>
+    <rightJoint>right_front_rev right_back_rev</rightJoint>
+    <wheelSeparation>0.64</wheelSeparation>
+    <wheelDiameter>0.4</wheelDiameter>
+    <wheelAcceleration>12.0</wheelAcceleration>
+    <commandTopic>cmd_vel</commandTopic>
+    <odometryTopic>odom</odometryTopic>
+    <odometryFrame>odom</odometryFrame>
+    <robotBaseFrame>base_link</robotBaseFrame>
+    <odometrySource>1</odometrySource>
+    <!-- Set to true to publish transforms for the wheel links, defaults to false -->
+    <publishWheelTF>true</publishWheelTF>
+    <!-- Maximum torque which the wheels can produce, in Nm, defaults to 5 Nm -->
+    <wheelTorque>20</wheelTorque>
+    <!-- Set to true to swap right and left wheels, defaults to true -->
+    <legacyMode>false</legacyMode>
+  </plugin>
+</gazebo>
+<!-- friction -->
+<xacro:macro name="wheel_friction" params="name">
+  <gazebo reference="${name}">
+    <mu1>1.0</mu1>
+    <mu2>1.0</mu2>
+    <joint><provideFeedback>true</provideFeedback></joint>
+  </gazebo>
+</xacro:macro>
+<xacro:wheel_friction name="left_front"/>
+<xacro:wheel_friction name="left_back"/>
+<xacro:wheel_friction name="right_front"/>
+<xacro:wheel_friction name="right_back"/>
+<!-- tell ros to use the ros2 gazebo control package globally - placement shouldn't matter in file -->
+<gazebo>
+  <plugin name="gazebo_ros2_control" filename="libgazebo_ros2_control.so" />
+</gazebo>
 </robot>

Commit message: throwing hands with ros and gazebo (ros and gazebo are winning)

File: lunabot_description/urdf/dummy_bot.xacro (robot description, xacro)
@@ -5,8 +5,8 @@
 <xacro:property name="chassisLength" value="0.9"/>
 <xacro:property name="chassisWidth" value="0.5"/>
-<xacro:property name="chassisMass" value="50"/>
+<xacro:property name="chassisMass" value="50.0"/>
 <xacro:property name="wheelWidth" value="0.125"/>
 <xacro:property name="wheelRadius" value="0.2"/>
-<xacro:property name="wheelMass" value="5"/>
+<xacro:property name="wheelMass" value="5.0"/>
 <xacro:macro name="box_inertia" params="m x y z">
   <inertia  ixx="${m*(y*y+z*z)/12}" ixy = "0" ixz = "0"
@@ -127,30 +127,8 @@
   </transmission>
 </xacro:macro>
-<xacro:transmission joint_name="left_front_rev"/>
-<xacro:transmission joint_name="left_back_rev"/>
-<xacro:transmission joint_name="right_front_rev"/>
-<xacro:transmission joint_name="right_back_rev"/>
-<!-- diff drive controller in gazebo -->
-<gazebo reference="base_link">
-  <plugin name="diff_drive_controller" filename="libgazebo_ros_diff_drive.so">
-    <updateRate>60</updateRate>
-    <leftJoint>left_front_rev left_back_rev</leftJoint>
-    <rightJoint>right_front_rev right_back_rev</rightJoint>
-    <wheelSeparation>0.64</wheelSeparation>
-    <wheelDiameter>0.4</wheelDiameter>
-    <wheelAcceleration>12.0</wheelAcceleration>
-    <commandTopic>cmd_vel</commandTopic>
-    <odometryTopic>odom</odometryTopic>
-    <odometryFrame>odom</odometryFrame>
-    <robotBaseFrame>base_link</robotBaseFrame>
-    <odometrySource>1</odometrySource>
-    <!-- Set to true to publish transforms for the wheel links, defaults to false -->
-    <publishWheelTF>true</publishWheelTF>
-    <!-- Maximum torque which the wheels can produce, in Nm, defaults to 5 Nm -->
-    <wheelTorque>20</wheelTorque>
-    <!-- Set to true to swap right and left wheels, defaults to true -->
-    <legacyMode>false</legacyMode>
-  </plugin>
-</gazebo>
+<!-- <xacro:transmission joint_name="left_front_rev"/> -->
+<!-- <xacro:transmission joint_name="left_back_rev"/> -->
+<!-- <xacro:transmission joint_name="right_front_rev"/> -->
+<!-- <xacro:transmission joint_name="right_back_rev"/> -->
 <!-- friction -->
 <xacro:macro name="wheel_friction" params="name">
@@ -161,11 +139,12 @@
   </gazebo>
 </xacro:macro>
-<xacro:wheel_friction name="left_front"/>
-<xacro:wheel_friction name="left_back"/>
-<xacro:wheel_friction name="right_front"/>
-<xacro:wheel_friction name="right_back"/>
-<!-- tell ros to use the ros2 gazebo control package globally - placement shouldn't matter in file -->
+<!-- <xacro:wheel_friction name="left_front"/> -->
+<!-- <xacro:wheel_friction name="left_back"/> -->
+<!-- <xacro:wheel_friction name="right_front"/> -->
+<!-- <xacro:wheel_friction name="right_back"/> -->
 <gazebo>
-  <plugin name="gazebo_ros2_control" filename="libgazebo_ros2_control.so" />
+  <plugin filename="libgazebo_ros2_control.so" name="gazebo_ros2_control">
+    <parameters>$(find mining_arena_gazebo)/config/diff_drive_controller.yaml</parameters>
+  </plugin>
 </gazebo>
 </robot>
