Commit message: Errors, Yay!

File: lunabot_description/urdf/bot.xacro.urdf (robot description, URDF)
Before this commit: robot dummy_bot, 5 links, 4 joints
Links:
- added link d455_back_bottom_screw_frame; collision mesh filename=package://chiconybot_description/meshes/sensors/d435.dae; visual mesh filename=package://chiconybot_description/meshes/sensors/d435.dae
- added link d455_back_color_frame
- added link d455_back_color_optical_frame
- added link d455_back_depth_frame
- added link d455_back_depth_optical_frame
- added link d455_back_left_ir_frame
- added link d455_back_left_ir_optical_frame
- added link d455_back_link
- added link d455_back_right_ir_frame
- added link d455_back_right_ir_optical_frame
- added link realsense_link; collision box ; visual mesh 
Joints:
- added joint d455_back_color_joint: type fixed, parent d455_back_depth_frame, child d455_back_color_frame
- added joint d455_back_color_optical_joint: type fixed, parent d455_back_color_frame, child d455_back_color_optical_frame
- added joint d455_back_depth_joint: type fixed, parent d455_back_link, child d455_back_depth_frame
- added joint d455_back_depth_optical_joint: type fixed, parent d455_back_depth_frame, child d455_back_depth_optical_frame
- added joint d455_back_joint: type fixed, parent base_link, child d455_back_bottom_screw_frame
- added joint d455_back_left_ir_joint: type fixed, parent d455_back_depth_frame, child d455_back_left_ir_frame
- added joint d455_back_left_ir_optical_joint: type fixed, parent d455_back_left_ir_frame, child d455_back_left_ir_optical_frame
- added joint d455_back_link_joint: type fixed, parent d455_back_bottom_screw_frame, child d455_back_link
- added joint d455_back_right_ir_joint: type fixed, parent d455_back_depth_frame, child d455_back_right_ir_frame
- added joint d455_back_right_ir_optical_joint: type fixed, parent d455_back_right_ir_frame, child d455_back_right_ir_optical_frame
- added joint realsense_joint: type fixed, parent , child 

Commit message: more changes

File: lunabot_description/urdf/bot.xacro.urdf (robot description, URDF)
Before this commit: robot dummy_bot, 16 links, 15 joints
Links:
- removed link d455_back_bottom_screw_frame
- removed link d455_back_color_frame
- removed link d455_back_color_optical_frame
- removed link d455_back_depth_frame
- removed link d455_back_depth_optical_frame
- removed link d455_back_left_ir_frame
- removed link d455_back_left_ir_optical_frame
- removed link d455_back_link
- removed link d455_back_right_ir_frame
- removed link d455_back_right_ir_optical_frame
- removed link realsense_link
Joints:
- removed joint d455_back_color_joint
- removed joint d455_back_color_optical_joint
- removed joint d455_back_depth_joint
- removed joint d455_back_depth_optical_joint
- removed joint d455_back_joint
- removed joint d455_back_left_ir_joint
- removed joint d455_back_left_ir_optical_joint
- removed joint d455_back_link_joint
- removed joint d455_back_right_ir_joint
- removed joint d455_back_right_ir_optical_joint
- removed joint realsense_joint

Commit message: new gazebo + robot model

File: lunabot_description/urdf/bot.xacro.urdf (robot description, URDF)
Before this commit: robot dummy_bot, 5 links, 4 joints
Links:
- link base_link: geometry collision mesh filename=model://realistic_robot/realistic_robot.stl; visual mesh filename=model://realistic_robot/realistic_robot.stl
- link left_back: geometry collision mesh filename=model://realistic_robot/robot_wheel.stl; visual mesh filename=model://realistic_robot/robot_wheel.stl
- link left_front: geometry collision mesh filename=model://realistic_robot/robot_wheel.stl; visual mesh filename=model://realistic_robot/robot_wheel.stl
- link right_back: geometry collision mesh filename=model://realistic_robot/robot_wheel.stl; visual mesh filename=model://realistic_robot/robot_wheel.stl
- link right_front: geometry collision mesh filename=model://realistic_robot/robot_wheel.stl; visual mesh filename=model://realistic_robot/robot_wheel.stl
Joints:
- joint left_back_rev: origin xyz=-0.25 0.32 0 rpy=0 0 0 -> xyz=0.217 -0.35 -0.162 rpy=0 0 0
- joint left_front_rev: origin xyz=0.25 0.32 0 rpy=0 0 0 -> xyz=-0.292 -0.35 -0.162 rpy=0 0 0
- joint right_back_rev: origin xyz=-0.25 -0.32 0 rpy=0 0 0 -> xyz=0.217 0.22 -0.162 rpy=0 0 0
- joint right_front_rev: origin xyz=0.25 -0.32 0 rpy=0 0 0 -> xyz=-0.292 0.22 -0.162 rpy=0 0 0

Commit message: everything except cmd_vel works

File: lunabot_description/urdf/bot.xacro.urdf (robot description, URDF)
Before this commit: robot dummy_bot, 5 links, 4 joints
Links:
- added link d455_back_depth_link
- added link d455_back_link, mass 0.035; collision box size=0.03 0.1 0.03; visual box size=0.03 0.1 0.03
- added link d455_back_rgb_link
- added link d455_front_depth_link
- added link d455_front_link, mass 0.035; collision box size=0.03 0.1 0.03; visual box size=0.03 0.1 0.03
- added link d455_front_rgb_link
- link base_link: geometry collision mesh filename=file://$(find mining_arena_gazebo)/models/realistic_robot/r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; visual mesh filename=file://$(find mining_arena_gazebo)/models/realistic_robot/r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
- link left_back: geometry collision mesh filename=file://$(find mining_arena_gazebo)/models/realistic_robot/r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; visual mesh filename=file://$(find mining_arena_gazebo)/models/realistic_robot/r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
- link left_front: geometry collision mesh filename=file://$(find mining_arena_gazebo)/models/realistic_robot/r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; visual mesh filename=file://$(find mining_arena_gazebo)/models/realistic_robot/r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
- link right_back: geometry collision mesh filename=file://$(find mining_arena_gazebo)/models/realistic_robot/r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; visual mesh filename=file://$(find mining_arena_gazebo)/models/realistic_robot/r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
- link right_front: geometry collision mesh filename=file://$(find mining_arena_gazebo)/models/realistic_robot/r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; visual mesh filename=file://$(find mining_arena_gazebo)/models/realistic_robot/r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
Joints:
- added joint d455_back_depth_joint: type fixed, parent d455_back_link, child d455_back_depth_link, origin xyz=0 0 0 rpy=${-pi/2} 0 ${-pi/2}
- added joint d455_back_joint: type fixed, parent base_link, child d455_back_link, origin xyz=0.39 -0.05 0.215 rpy=0 0 0, axis 0 0 1
- added joint d455_back_rgb_joint: type fixed, parent d455_back_link, child d455_back_rgb_link, origin xyz=0 0 0 rpy=${-pi/2} 0 ${-pi/2}
- added joint d455_front_depth_joint: type fixed, parent d455_front_link, child d455_front_depth_link, origin xyz=0 0 0 rpy=${-pi/2} 0 ${-pi/2}
- added joint d455_front_joint: type fixed, parent base_link, child d455_front_link, origin xyz=-0.55 0.15 0 rpy=0 0 3.1415, axis 0 0 1
- added joint d455_front_rgb_joint: type fixed, parent d455_front_link, child d455_front_rgb_link, origin xyz=0 0 0 rpy=${-pi/2} 0 ${-pi/2}

Commit message: ros2 sim conversion complete

File: lunabot_description/urdf/bot.xacro.urdf (robot description, URDF)
Before this commit: robot dummy_bot, 11 links, 10 joints
Links:
- added link middle_link
Joints:
- added joint mid_joint: type fixed, parent base_link, child middle_link, origin xyz=0 0 0 rpy=0 0 3.14, axis 0 0 1
- joint d455_back_joint: parent base_link -> middle_link
- joint d455_front_joint: origin xyz=-0.55 0.15 0 rpy=0 0 3.1415 -> xyz=-0.55 0.15 0 rpy=0 0 3.14; parent base_link -> middle_link
- joint left_back_rev: parent base_link -> middle_link
- joint left_front_rev: parent base_link -> middle_link
- joint right_back_rev: parent base_link -> middle_link
- joint right_front_rev: parent base_link -> middle_link

Commit message: no more cool model

File: lunabot_description/urdf/bot.xacro.urdf (robot description, URDF)
Before this commit: robot dummy_bot, 12 links, 11 joints
Links:
- link base_link: geometry collision box size=0.9 0.5 0.1; visual box size=0.9 0.5 0.1
- link left_back: geometry collision cylinder length=0.125 radius=0.2; visual cylinder length=0.125 radius=0.2
- link left_front: geometry collision cylinder length=0.125 radius=0.2; visual cylinder length=0.125 radius=0.2
- link right_back: geometry collision cylinder length=0.125 radius=0.2; visual cylinder length=0.125 radius=0.2
- link right_front: geometry collision cylinder length=0.125 radius=0.2; visual cylinder length=0.125 radius=0.2

Commit message: refactor mining_arena_gazebo to lunabot_sim

File: lunabot_description/urdf/bot.xacro.urdf (robot description, URDF)
Before this commit: robot dummy_bot, 12 links, 11 joints
Links:
- link base_link: geometry collision mesh filename=file://$(find lunabot_sim)/models/realistic_robot/realistic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; visual mesh filename=file://$(find lunabot_sim)/models/realistic_robot/realistic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
- link left_back: geometry collision mesh filename=file://$(find lunabot_sim)/models/realistic_robot/robot_whe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; visual mesh filename=file://$(find lunabot_sim)/models/realistic_robot/robot_whe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
- link left_front: geometry collision mesh filename=file://$(find lunabot_sim)/models/realistic_robot/robot_whe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; visual mesh filename=file://$(find lunabot_sim)/models/realistic_robot/robot_whe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
- link right_back: geometry collision mesh filename=file://$(find lunabot_sim)/models/realistic_robot/robot_whe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; visual mesh filename=file://$(find lunabot_sim)/models/realistic_robot/robot_whe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
- link right_front: geometry collision mesh filename=file://$(find lunabot_sim)/models/realistic_robot/robot_whe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; visual mesh filename=file://$(find lunabot_sim)/models/realistic_robot/robot_whe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
