Commit message: add dummy bot and clean up files

File: lunabot_description/urdf/dummy_bot.xacro.urdf (robot description, URDF)
Before this commit: robot dummy_bot, 1 links, 0 joints
Links:
- added link d455_back_depth_link
- added link d455_back_link, mass 0.035; collision box size=0.03 0.1 0.03; visual box size=0.03 0.1 0.03
- added link d455_back_rgb_link
- added link d455_front_depth_link
- added link d455_front_link, mass 0.035; collision box size=0.03 0.1 0.03; visual box size=0.03 0.1 0.03
- added link d455_front_rgb_link
- added link left_back, mass 5.0; collision cylinder length=0.125 radius=0.2; visual cylinder length=0.125 radius=0.2
- added link left_front, mass 5.0; collision cylinder length=0.125 radius=0.2; visual cylinder length=0.125 radius=0.2
- added link middle_link
- added link right_back, mass 5.0; collision cylinder length=0.125 radius=0.2; visual cylinder length=0.125 radius=0.2
- added link right_front, mass 5.0; collision cylinder length=0.125 radius=0.2; visual cylinder length=0.125 radius=0.2
- link base_link: mass ${chassisMass} -> 50.0; geometry collision box size=0.9 0.5 0.1; visual box size=0.9 0.5 0.1
Joints:
- added joint d455_back_depth_joint: type fixed, parent d455_back_link, child d455_back_depth_link, origin xyz=0 0 0 rpy=${-pi/2} 0 ${-pi/2}
- added joint d455_back_joint: type fixed, parent middle_link, child d455_back_link, origin xyz=0.39 -0.05 0.215 rpy=0 0 0, axis 0 0 1
- added joint d455_back_rgb_joint: type fixed, parent d455_back_link, child d455_back_rgb_link, origin xyz=0 0 0 rpy=${-pi/2} 0 ${-pi/2}
- added joint d455_front_depth_joint: type fixed, parent d455_front_link, child d455_front_depth_link, origin xyz=0 0 0 rpy=${-pi/2} 0 ${-pi/2}
- added joint d455_front_joint: type fixed, parent middle_link, child d455_front_link, origin xyz=-0.55 0.15 0 rpy=0 0 3.14, axis 0 0 1
- added joint d455_front_rgb_joint: type fixed, parent d455_front_link, child d455_front_rgb_link, origin xyz=0 0 0 rpy=${-pi/2} 0 ${-pi/2}
- added joint left_back_rev: type continuous, parent middle_link, child left_back, origin xyz=0.217 -0.35 -0.162 rpy=0 0 0, axis 0 1 0
- added joint left_front_rev: type continuous, parent middle_link, child left_front, origin xyz=-0.292 -0.35 -0.162 rpy=0 0 0, axis 0 1 0
- added joint mid_joint: type fixed, parent base_link, child middle_link, origin xyz=0 0 0 rpy=0 0 3.14, axis 0 0 1
- added joint right_back_rev: type continuous, parent middle_link, child right_back, origin xyz=0.217 0.22 -0.162 rpy=0 0 0, axis 0 1 0
- added joint right_front_rev: type continuous, parent middle_link, child right_front, origin xyz=-0.292 0.22 -0.162 rpy=0 0 0, axis 0 1 0

Commit message: remove computation stuff from sim

File: lunabot_description/urdf/dummy_bot.xacro.urdf (robot description, URDF)
Before this commit: robot dummy_bot, 12 links, 11 joints
Links:
- removed link d455_back_depth_link
- removed link d455_back_link
- removed link d455_back_rgb_link
- removed link d455_front_depth_link
- removed link d455_front_link
- removed link d455_front_rgb_link
Joints:
- removed joint d455_back_depth_joint
- removed joint d455_back_joint
- removed joint d455_back_rgb_joint
- removed joint d455_front_depth_joint
- removed joint d455_front_joint
- removed joint d455_front_rgb_joint

Commit message: Changed transforms to align with REP standards -- Isaac

File: lunabot_description/urdf/dummy_bot.xacro.urdf (robot description, URDF)
Before this commit: robot dummy_bot, 12 links, 11 joints
Joints:
- joint d455_back_joint: origin xyz=0.39 -0.05 0.215 rpy=0 0 0 -> xyz=-0.381 0.05 0.558 rpy=${pi} 0 ${pi}
- joint d455_front_joint: origin xyz=-0.55 0.15 0 rpy=0 0 3.14 -> xyz=0.558 -0.17 0.33 rpy=0 0.3 0
- joint left_back_rev: origin xyz=0.217 -0.35 -0.162 rpy=0 0 0 -> xyz=-0.228 0.254 0.178 rpy=0 0 0
- joint left_front_rev: origin xyz=-0.292 -0.35 -0.162 rpy=0 0 0 -> xyz=0.3302 0.254 0.1778 rpy=0 0 0
- joint mid_joint: origin xyz=0 0 0 rpy=0 0 3.14 -> xyz=0 0 0 rpy=0 0 0
- joint right_back_rev: origin xyz=0.217 0.22 -0.162 rpy=0 0 0 -> xyz=-0.228 -0.254 0.178 rpy=0 0 0
- joint right_front_rev: origin xyz=-0.292 0.22 -0.162 rpy=0 0 0 -> xyz=0.3302 -0.254 0.178 rpy=0 0 0

Commit message: Make manual control work
This does not actually rely on anything in the nav2 version of two
robot, it's just where I'm working

File: lunabot_description/urdf/dummy_bot.xacro.urdf (robot description, URDF)
Before this commit: robot dummy_bot, 12 links, 11 joints
Joints:
- joint d455_back_joint: origin xyz=-0.381 0.05 0.558 rpy=${pi} 0 ${pi} -> xyz=0.39 -0.05 0.215 rpy=0 0 0
- joint d455_front_joint: origin xyz=0.558 -0.17 0.33 rpy=0 0.3 0 -> xyz=-0.55 0.15 0 rpy=0 0 3.14
- joint left_back_rev: origin xyz=-0.228 0.254 0.178 rpy=0 0 0 -> xyz=0.217 -0.35 -0.162 rpy=0 0 0
- joint left_front_rev: origin xyz=0.3302 0.254 0.1778 rpy=0 0 0 -> xyz=-0.292 -0.35 -0.162 rpy=0 0 0
- joint mid_joint: origin xyz=0 0 0 rpy=0 0 0 -> xyz=0 0 0 rpy=0 0 3.14
- joint right_back_rev: origin xyz=-0.228 -0.254 0.178 rpy=0 0 0 -> xyz=0.217 0.22 -0.162 rpy=0 0 0
- joint right_front_rev: origin xyz=0.3302 -0.254 0.178 rpy=0 0 0 -> xyz=-0.292 0.22 -0.162 rpy=0 0 0

Commit message: Change transforms so sim and real bot work at the same time
Base link is the center of the robot on the floor

File: lunabot_description/urdf/dummy_bot.xacro.urdf (robot description, URDF)
Before this commit: robot dummy_bot, 12 links, 11 joints
Links:
- link base_link: mass 50.0 -> None; geometry 
- link middle_link: mass None -> 50.0; geometry collision box size=0.9 0.5 0.1; visual box size=0.9 0.5 0.1
Joints:
- joint d455_back_joint: parent middle_link -> base_link
- joint d455_front_joint: parent middle_link -> base_link
- joint left_back_rev: parent middle_link -> base_link
- joint left_front_rev: parent middle_link -> base_link
- joint mid_joint: origin xyz=0 0 0 rpy=0 0 0 -> xyz=0.1 0 0.3 rpy=0 0 0
- joint right_back_rev: parent middle_link -> base_link
- joint right_front_rev: parent middle_link -> base_link

Commit message: Add excavation to sim and put the camera on it

File: lunabot_description/urdf/dummy_bot.xacro.urdf (robot description, URDF)
Before this commit: robot dummy_bot, 12 links, 11 joints
Links:
- added link excavation, mass 10.0; collision box size=0.75 0.13 0.1; visual box size=0.75 0.13 0.1
- link middle_link: mass 50.0 -> 40.0
Joints:
- added joint excavation_joint: type prismatic, parent middle_link, child excavation, origin xyz=0.4 0 0.2 rpy=0 -2.0944 0, axis 1 0 0, limit lower=-10 upper=10 effort=1000.0 velocity=0.5
- joint d455_front_joint: origin xyz=0.558 -0.17 0.33 rpy=0 0.3 0 -> xyz=0.3 -0.17 0.0 rpy=0 2.5 0; parent base_link -> excavation

Commit message: raytracing! now we need a 5090

File: lunabot_description/urdf/dummy_bot.xacro.urdf (robot description, URDF)
Before this commit: robot dummy_bot, 12 links, 11 joints
Joints:
- joint left_front_rev: origin xyz=0.3302 0.254 0.1778 rpy=0 0 0 -> xyz=0.3302 0.254 0.178 rpy=0 0 0

Commit message: add apriltag to sim

File: lunabot_description/urdf/dummy_bot.xacro.urdf (robot description, URDF)
Before this commit: robot dummy_bot, 12 links, 11 joints
Links:
- added link deposition_apriltag_link, mass 0.1; visual mesh filename=package://lunabot_sim/models/apriltag_dae/apriltag.dae scale=0.1524 0.1524 1
Joints:
- added joint deposition_apriltag_joint: type fixed, parent base_link, child deposition_apriltag_link, origin xyz=-0.381 0.0 0.5 rpy=0.0 -0.34 3.14
- joint d455_back_joint: origin xyz=-0.381 0.05 0.558 rpy=${pi} 0 ${pi} -> xyz=-0.44 0.0 0.65 rpy=0 0.6 ${pi}
- joint mid_joint: axis 0 0 1 -> (none); origin xyz=0.1 0 0.3 rpy=0 0 0 -> xyz=0.0 0 0.3 rpy=0 0 0

Commit message: adjust camera frames

File: lunabot_description/urdf/dummy_bot.xacro.urdf (robot description, URDF)
Before this commit: robot dummy_bot, 14 links, 13 joints
Joints:
- joint d455_front_joint: origin xyz=0.3 -0.17 0.0 rpy=0 2.5 0 -> xyz=0.3 0.17 0.0 rpy=0 2.5 0

File: lunabot_description/urdf/mini_bot.xacro.urdf (robot description, URDF)
Before this commit: robot mini_bot, 12 links, 11 joints
Joints:
- joint d455_back_joint: origin xyz=-0.381 0.05 0.558 rpy=${pi} 0 ${pi} -> xyz=-0.21 0 0.5 rpy=0 0 ${pi}
- joint d455_front_joint: origin xyz=0.558 -0.17 0.33 rpy=0 0.3 0 -> xyz=0.2 0 0.5 rpy=0 0.5 0
- joint mid_joint: axis 0 0 1 -> (none)

Commit message: fixing some lidar issues

File: lunabot_description/urdf/dummy_bot.xacro.urdf (robot description, URDF)
Before this commit: robot dummy_bot, 12 links, 11 joints
Links:
- added link lidar_link, mass 0.035; collision box size=0.03 0.1 0.03; visual box size=0.03 0.1 0.03
Joints:
- added joint lidar_joint: type fixed, parent base_link, child lidar_link, origin xyz=-0.381 -0.05 0.558 rpy=${pi} 0 ${pi}, axis 0 0 1

Commit message: Connect effort to sim excavation actuators
- Also publish rough current

File: lunabot_description/urdf/dummy_bot.xacro.urdf (robot description, URDF)
Before this commit: robot dummy_bot, 14 links, 13 joints
Joints:
- joint excavation_joint: limit lower=-10 upper=10 effort=1000.0 velocity=0.5 -> lower=-0.2 upper=0.0 effort=1000.0 velocity=0.5

Commit message: lidar mostly works, need to fix transforms

File: lunabot_description/urdf/dummy_bot.xacro.urdf (robot description, URDF)
Before this commit: robot dummy_bot, 13 links, 12 joints
Links:
- added link lidar_mid_link
- link lidar_link: mass 0.035 -> None; geometry 
Joints:
- added joint lidar_joint2: type fixed, parent lidar_mid_link, child lidar_link, origin xyz=0 0 0 rpy=0 0 ${pi*0.375}, axis 0 0 1
- joint lidar_joint: child lidar_link -> lidar_mid_link; origin xyz=-0.381 -0.05 0.558 rpy=${pi} 0 ${pi} -> xyz=-0.381 -0.05 0.558 rpy=0 ${-pi/2} 0

Commit message: Changed from sandpit testing 2/28x

File: lunabot_description/urdf/dummy_bot.xacro.urdf (robot description, URDF)
Before this commit: robot dummy_bot, 14 links, 13 joints
Links:
- removed link deposition_apriltag_link
- removed link excavation
- link middle_link: mass 40.0 -> 50.0
Joints:
- removed joint deposition_apriltag_joint
- removed joint excavation_joint
- joint d455_back_joint: origin xyz=-0.44 0.0 0.65 rpy=0 0.6 ${pi} -> xyz=-0.381 0.05 0.558 rpy=${pi} 0 ${pi}
- joint d455_front_joint: origin xyz=0.3 0.17 0.0 rpy=0 2.5 0 -> xyz=0.558 -0.17 0.33 rpy=0 0.4712 0; parent excavation -> base_link
- joint mid_joint: axis (none) -> 0 0 1; origin xyz=0.0 0 0.3 rpy=0 0 0 -> xyz=0.1 0 0.3 rpy=0 0 0

Commit message: add deposition apriltag optical frame

File: lunabot_description/urdf/dummy_bot.xacro.urdf (robot description, URDF)
Before this commit: robot dummy_bot, 14 links, 13 joints
Links:
- added link deposition_apriltag_optical_frame
Joints:
- added joint deposition_apriltag_optical_joint: type fixed, parent deposition_apriltag_link, child deposition_apriltag_optical_frame, origin xyz=0.0 0.0 0.0 rpy=1.57 0.0 1.57

Commit message: fix urdfs

File: lunabot_description/urdf/dummy_bot.xacro.urdf (robot description, URDF)
Before this commit: robot dummy_bot, 15 links, 14 joints
Joints:
- joint d455_front_joint: origin xyz=0.3 0.17 0.0 rpy=0 2.5 0 -> xyz=0.3 -0.17 0.0 rpy=0 2.5 0

File: lunabot_description/urdf/mini_bot.xacro.urdf (robot description, URDF)
Before this commit: robot mini_bot, 12 links, 11 joints
Joints:
- joint d455_back_joint: origin xyz=-0.21 0 0.5 rpy=0 0 ${pi} -> xyz=-0.155 0 0.42953 rpy=0 0 ${pi}; parent base_link -> middle_link
- joint d455_front_joint: origin xyz=0.2 0 0.5 rpy=0 0.5 0 -> xyz=0.18939 0.16173 0.428 rpy=0 0.5 0; parent base_link -> middle_link

Commit message: Move apriltag up a little bit

File: lunabot_description/urdf/dummy_bot.xacro.urdf (robot description, URDF)
Before this commit: robot dummy_bot, 15 links, 14 joints
Joints:
- joint deposition_apriltag_joint: origin xyz=-0.381 0.0 0.5 rpy=0.0 -0.34 3.14 -> xyz=-0.381 0.0 0.55 rpy=0.0 -0.34 3.14

Commit message: fix record and tfs

File: lunabot_description/urdf/dummy_bot.xacro.urdf (robot description, URDF)
Before this commit: robot dummy_bot, 17 links, 16 joints
Links:
- removed link lidar_link
- removed link lidar_mid_link
Joints:
- removed joint lidar_joint
- removed joint lidar_joint2

File: lunabot_description/urdf/mini_bot.xacro.urdf (robot description, URDF)
Before this commit: robot mini_bot, 12 links, 11 joints
Links:
- added link lidar_link
- added link lidar_mid_link
Joints:
- added joint lidar_joint: type fixed, parent lidar_mid_link, child lidar_link, origin xyz=0 0 0 rpy=0 0 ${pi*0.375}, axis 0 0 1
- added joint lidar_mid_joint: type fixed, parent base_link, child lidar_mid_link, origin xyz=0.18939 -0.51 0.44 rpy=0 ${-pi/2} 0, axis 0 0 1
- joint d455_front_joint: origin xyz=0.18939 0.16173 0.428 rpy=${pi} 0.523599 0 -> xyz=0.18939 0.16173 0.428 rpy=0 0.523599 0

Commit message: Changes from real life testing

File: lunabot_description/urdf/dummy_bot.xacro.urdf (robot description, URDF)
Before this commit: robot dummy_bot, 15 links, 14 joints
Joints:
- joint d455_back_joint: origin xyz=-0.44 0.0 0.65 rpy=0 0.6 ${pi} -> xyz=-0.44 0.0 0.65 rpy=${pi} 0.7 ${pi}
- joint d455_front_joint: origin xyz=0.3 -0.17 0.0 rpy=0 2.5 0 -> xyz=0.3 -0.17 0.0 rpy=${pi} ${-0.55 + pi} 0

Commit message: Update apriltags on the main for the small and big tags

File: lunabot_description/urdf/dummy_bot.xacro.urdf (robot description, URDF)
Before this commit: robot dummy_bot, 15 links, 14 joints
Links:
- added link deposition_apriltag_small_link
- added link deposition_apriltag_small_optical_frame
Joints:
- added joint deposition_apriltag_small_joint: type fixed, parent base_link, child deposition_apriltag_small_link, origin xyz=-0.381 0.15 0.55 rpy=0.0 -0.34 3.14
- added joint deposition_apriltag_small_optical_joint: type fixed, parent deposition_apriltag_small_link, child deposition_apriltag_small_optical_frame, origin xyz=0.0 0.0 0.0 rpy=1.57 0.0 1.57
- joint deposition_apriltag_joint: origin xyz=-0.381 0.0 0.55 rpy=0.0 -0.34 3.14 -> xyz=-0.381 -0.03 0.55 rpy=0.0 -0.34 3.14

Commit message: second starting zone apriltag

File: lunabot_description/urdf/dummy_bot.xacro.urdf (robot description, URDF)
Before this commit: robot dummy_bot, 17 links, 16 joints
Joints:
- joint d455_front_joint: origin xyz=0.3 -0.17 0.0 rpy=${pi} ${-0.55 + pi} 0 -> xyz=0.3 -0.17 0.0 rpy=0 ${-0.67 + pi} 0

Commit message: WIP changing sim apriltags

File: lunabot_description/urdf/dummy_bot.xacro.urdf (robot description, URDF)
Before this commit: robot dummy_bot, 17 links, 16 joints
Links:
- link deposition_apriltag_link: geometry visual mesh filename=package://lunabot_sim/models/apriltag_126_dae/apriltag.dae scale=0.12 0.12 1
- link deposition_apriltag_small_link: mass None -> 0.1; geometry visual mesh filename=package://lunabot_sim/models/apriltag_173_dae/apriltag.dae scale=0.025 0.025 1

Commit message: add deposition apriltags in sim - Isaac

File: lunabot_description/urdf/dummy_bot.xacro.urdf (robot description, URDF)
Before this commit: robot dummy_bot, 17 links, 16 joints
Links:
- link deposition_apriltag_link: geometry visual mesh filename=package://lunabot_sim/models/apriltag_126_dae/apriltag_126.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 scale=0.12 0.12 1
- link deposition_apriltag_small_link: geometry visual mesh filename=package://lunabot_sim/models/apriltag_173_dae/apriltag_173.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 scale=0.025 0.025 1
Joints:
- joint d455_back_joint: origin xyz=-0.44 0.0 0.65 rpy=${pi} 0.7 ${pi} -> xyz=-0.44 0.02 0.63 rpy=${pi} 0.7 ${pi}
- joint deposition_apriltag_joint: origin xyz=-0.381 -0.03 0.55 rpy=0.0 -0.34 3.14 -> xyz=-0.42 -0.02 0.51 rpy=0.0 -0.35 3.14
- joint deposition_apriltag_small_joint: origin xyz=-0.381 0.15 0.55 rpy=0.0 -0.34 3.14 -> xyz=-0.42 0.09 0.51 rpy=0.0 -0.35 3.14

File: lunabot_description/urdf/mini_bot.xacro.urdf (robot description, URDF)
Before this commit: robot mini_bot, 14 links, 13 joints
Joints:
- joint d455_back_joint: origin xyz=-0.155 0 0.42953 rpy=0 0 ${pi} -> xyz=-0.155 0 0.51 rpy=0 0 ${pi}; parent middle_link -> base_link
- joint d455_front_joint: origin xyz=0.18939 0.16173 0.428 rpy=0 0.523599 0 -> xyz=0.18939 0.16173 0.52 rpy=0 0.523599 0; parent middle_link -> base_link

Commit message: new camera mount

File: lunabot_description/urdf/dummy_bot.xacro.urdf (robot description, URDF)
Before this commit: robot dummy_bot, 17 links, 16 joints
Joints:
- joint d455_front_joint: origin xyz=0.3 -0.17 0.0 rpy=0 ${-0.67 + pi} 0 -> xyz=0.3 0.0 -0.15 rpy=0 ${-0.663 + pi} 0

Commit message: Add very basic mujoco sim

File: lunabot_description/urdf/dummy_bot.xacro.urdf (robot description, URDF)
Before this commit: robot dummy_bot, 17 links, 16 joints
Links:
- removed link d455_back_depth_link
- removed link d455_back_rgb_link
- removed link d455_front_depth_link
- removed link d455_front_rgb_link
- added link d455_back_sim_link
- added link d455_front_sim_link
- link d455_back_link: mass 0.035 -> None; geometry visual box size=0.03 0.1 0.03
- link d455_front_link: mass 0.035 -> None; geometry visual box size=0.03 0.1 0.03
- link deposition_apriltag_link: mass 0.1 -> None
- link deposition_apriltag_small_link: mass 0.1 -> None
- link excavation: mass 10.0 -> None; geometry visual box size=0.75 0.13 0.1
- link left_back: mass 5.0 -> None; geometry visual cylinder length=0.125 radius=0.2
- link left_front: mass 5.0 -> None; geometry visual cylinder length=0.125 radius=0.2
- link middle_link: mass 40.0 -> None; geometry visual box size=0.9 0.5 0.1
- link right_back: mass 5.0 -> None; geometry visual cylinder length=0.125 radius=0.2
- link right_front: mass 5.0 -> None; geometry visual cylinder length=0.125 radius=0.2
Joints:
- removed joint d455_back_depth_joint
- removed joint d455_back_rgb_joint
- removed joint d455_front_depth_joint
- removed joint d455_front_rgb_joint
- added joint d455_back_sim_joint: type fixed, parent d455_back_link, child d455_back_sim_link, origin xyz=0 0 0 rpy=${pi/2} 0 ${pi/2}
- added joint d455_front_sim_joint: type fixed, parent d455_front_link, child d455_front_sim_link, origin xyz=0 0 0 rpy=${pi/2} 0 ${pi/2}
- joint d455_front_joint: axis 0 0 1 -> (none)
- joint excavation_joint: type prismatic -> fixed

Commit message: Finish mujoco sim
Except for rocks and stuff, which is easy

File: lunabot_description/urdf/dummy_bot.xacro.urdf (robot description, URDF)
Before this commit: robot dummy_bot, 15 links, 14 joints
Joints:
- joint excavation_joint: type fixed -> prismatic
