Commit message: Fix the mini bot urdf and remove nav2 controller test stuff

File: lunabot_description/urdf/mini_bot.xacro.urdf (robot description, URDF)
Before this commit: robot mini_bot, 12 links, 11 joints
Links:
- link base_link: mass 50.0 -> None; geometry 
- link middle_link: mass None -> 50.0; geometry collision box size=0.9 0.5 0.1; visual box size=0.9 0.5 0.1
Joints:
- joint d455_back_joint: origin xyz=0.39 -0.05 0.215 rpy=0 0 0 -> xyz=-0.381 0.05 0.558 rpy=${pi} 0 ${pi}; parent middle_link -> base_link
- joint d455_front_joint: origin xyz=-0.55 0.15 0 rpy=0 0 3.14 -> xyz=0.558 -0.17 0.33 rpy=0 0.3 0; parent middle_link -> base_link
- joint left_back_rev: origin xyz=0.217 -0.35 -0.162 rpy=0 0 0 -> xyz=-0.228 0.254 0.178 rpy=0 0 0; parent middle_link -> base_link
- joint left_front_rev: origin xyz=-0.292 -0.35 -0.162 rpy=0 0 0 -> xyz=0.3302 0.254 0.1778 rpy=0 0 0; parent middle_link -> base_link
- joint mid_joint: origin xyz=0 0 0 rpy=0 0 3.14 -> xyz=0.1 0 0.3 rpy=0 0 0
- joint right_back_rev: origin xyz=0.217 0.22 -0.162 rpy=0 0 0 -> xyz=-0.228 -0.254 0.178 rpy=0 0 0; parent middle_link -> base_link
- joint right_front_rev: origin xyz=-0.292 0.22 -0.162 rpy=0 0 0 -> xyz=0.3302 -0.254 0.178 rpy=0 0 0; parent middle_link -> base_link

Commit message: Make the mini bot correct
- Also fix some crashes on shutdown

File: lunabot_description/urdf/mini_bot.xacro.urdf (robot description, URDF)
Before this commit: robot mini_bot, 12 links, 11 joints
Links:
- link left_back: geometry collision cylinder length=0.09 radius=0.03; visual cylinder length=0.09 radius=0.03
- link left_front: geometry collision cylinder length=0.09 radius=0.03; visual cylinder length=0.09 radius=0.03
- link middle_link: geometry collision box size=0.355 0.43 0.1; visual box size=0.355 0.43 0.1
- link right_back: geometry collision cylinder length=0.09 radius=0.03; visual cylinder length=0.09 radius=0.03
- link right_front: geometry collision cylinder length=0.09 radius=0.03; visual cylinder length=0.09 radius=0.03
Joints:
- joint left_back_rev: origin xyz=-0.228 0.254 0.178 rpy=0 0 0 -> xyz=-0.2008 0.305 0.03 rpy=0 0 0
- joint left_front_rev: origin xyz=0.3302 0.254 0.1778 rpy=0 0 0 -> xyz=0.0532 0.305 0.03 rpy=0 0 0
- joint mid_joint: origin xyz=0.1 0 0.3 rpy=0 0 0 -> xyz=0.0 0 0.15 rpy=0 0 0
- joint right_back_rev: origin xyz=-0.228 -0.254 0.178 rpy=0 0 0 -> xyz=-0.2008 -0.305 0.03 rpy=0 0 0
- joint right_front_rev: origin xyz=0.3302 -0.254 0.178 rpy=0 0 0 -> xyz=0.0532 -0.305 0.03 rpy=0 0 0

Commit message: fix firmware and cameras

File: lunabot_description/urdf/mini_bot.xacro.urdf (robot description, URDF)
Before this commit: robot mini_bot, 12 links, 11 joints
Links:
- removed link base_link
- removed link d455_back_depth_link
- removed link d455_back_link
- removed link d455_back_rgb_link
- removed link d455_front_depth_link
- removed link d455_front_link
- removed link d455_front_rgb_link
- removed link left_back
- removed link left_front
- removed link middle_link
- removed link right_back
- removed link right_front
- added link mini/base_link
- added link mini/left_back, mass 5.0; collision cylinder length=0.09 radius=0.03; visual cylinder length=0.09 radius=0.03
- added link mini/left_front, mass 5.0; collision cylinder length=0.09 radius=0.03; visual cylinder length=0.09 radius=0.03
- added link mini/middle_link, mass 50.0; collision box size=0.355 0.43 0.1; visual box size=0.355 0.43 0.1
- added link mini/right_back, mass 5.0; collision cylinder length=0.09 radius=0.03; visual cylinder length=0.09 radius=0.03
- added link mini/right_front, mass 5.0; collision cylinder length=0.09 radius=0.03; visual cylinder length=0.09 radius=0.03
- added link mini_d455_back_depth_link
- added link mini_d455_back_link, mass 0.035; collision box size=0.03 0.1 0.03; visual box size=0.03 0.1 0.03
- added link mini_d455_back_rgb_link
- added link mini_d455_front_depth_link
- added link mini_d455_front_link, mass 0.035; collision box size=0.03 0.1 0.03; visual box size=0.03 0.1 0.03
- added link mini_d455_front_rgb_link
Joints:
- removed joint d455_back_depth_joint
- removed joint d455_back_joint
- removed joint d455_back_rgb_joint
- removed joint d455_front_depth_joint
- removed joint d455_front_joint
- removed joint d455_front_rgb_joint
- removed joint left_back_rev
- removed joint left_front_rev
- removed joint mid_joint
- removed joint right_back_rev
- removed joint right_front_rev
- added joint mini/left_back_rev: type continuous, parent mini/base_link, child mini/left_back, origin xyz=-0.2008 0.305 0.03 rpy=0 0 0, axis 0 1 0
- added joint mini/left_front_rev: type continuous, parent mini/base_link, child mini/left_front, origin xyz=0.0532 0.305 0.03 rpy=0 0 0, axis 0 1 0
- added joint mini/mid_joint: type fixed, parent mini/base_link, child mini/middle_link, origin xyz=0.0 0 0.15 rpy=0 0 0
- added joint mini/right_back_rev: type continuous, parent mini/base_link, child mini/right_back, origin xyz=-0.2008 -0.305 0.03 rpy=0 0 0, axis 0 1 0
- added joint mini/right_front_rev: type continuous, parent mini/base_link, child mini/right_front, origin xyz=0.0532 -0.305 0.03 rpy=0 0 0, axis 0 1 0
- added joint mini_d455_back_depth_joint: type fixed, parent mini_d455_back_link, child mini_d455_back_depth_link, origin xyz=0 0 0 rpy=${-pi/2} 0 ${-pi/2}
- added joint mini_d455_back_joint: type fixed, parent mini/middle_link, child mini_d455_back_link, origin xyz=-0.155 0 0.42953 rpy=0 0 ${pi}, axis 0 0 1
- added joint mini_d455_back_rgb_joint: type fixed, parent mini_d455_back_link, child mini_d455_back_rgb_link, origin xyz=0 0 0 rpy=${-pi/2} 0 ${-pi/2}
- added joint mini_d455_front_depth_joint: type fixed, parent mini_d455_front_link, child mini_d455_front_depth_link, origin xyz=0 0 0 rpy=${-pi/2} 0 ${-pi/2}
- added joint mini_d455_front_joint: type fixed, parent mini/middle_link, child mini_d455_front_link, origin xyz=0.18939 0.16173 0.428 rpy=0 0.5 0, axis 0 0 1
- added joint mini_d455_front_rgb_joint: type fixed, parent mini_d455_front_link, child mini_d455_front_rgb_link, origin xyz=0 0 0 rpy=${-pi/2} 0 ${-pi/2}

Commit message: works

File: lunabot_description/urdf/mini_bot.xacro.urdf (robot description, URDF)
Before this commit: robot mini_bot, 12 links, 11 joints
Joints:
- joint mini_d455_front_joint: origin xyz=0.18939 0.16173 0.428 rpy=0 0.5 0 -> xyz=0.18939 0.16173 0.428 rpy=${pi} 0.523599 0

Commit message: Undo the changes to the camera transforms

File: lunabot_description/urdf/mini_bot.xacro.urdf (robot description, URDF)
Before this commit: robot mini_bot, 12 links, 11 joints
Links:
- removed link mini/base_link
- removed link mini/left_back
- removed link mini/left_front
- removed link mini/middle_link
- removed link mini/right_back
- removed link mini/right_front
- removed link mini_d455_back_depth_link
- removed link mini_d455_back_link
- removed link mini_d455_back_rgb_link
- removed link mini_d455_front_depth_link
- removed link mini_d455_front_link
- removed link mini_d455_front_rgb_link
- added link base_link
- added link d455_back_depth_link
- added link d455_back_link, mass 0.035; collision box size=0.03 0.1 0.03; visual box size=0.03 0.1 0.03
- added link d455_back_rgb_link
- added link d455_front_depth_link
- added link d455_front_link, mass 0.035; collision box size=0.03 0.1 0.03; visual box size=0.03 0.1 0.03
- added link d455_front_rgb_link
- added link left_back, mass 5.0; collision cylinder length=0.09 radius=0.03; visual cylinder length=0.09 radius=0.03
- added link left_front, mass 5.0; collision cylinder length=0.09 radius=0.03; visual cylinder length=0.09 radius=0.03
- added link middle_link, mass 50.0; collision box size=0.355 0.43 0.1; visual box size=0.355 0.43 0.1
- added link right_back, mass 5.0; collision cylinder length=0.09 radius=0.03; visual cylinder length=0.09 radius=0.03
- added link right_front, mass 5.0; collision cylinder length=0.09 radius=0.03; visual cylinder length=0.09 radius=0.03
Joints:
- removed joint mini/left_back_rev
- removed joint mini/left_front_rev
- removed joint mini/mid_joint
- removed joint mini/right_back_rev
- removed joint mini/right_front_rev
- removed joint mini_d455_back_depth_joint
- removed joint mini_d455_back_joint
- removed joint mini_d455_back_rgb_joint
- removed joint mini_d455_front_depth_joint
- removed joint mini_d455_front_joint
- removed joint mini_d455_front_rgb_joint
- added joint d455_back_depth_joint: type fixed, parent d455_back_link, child d455_back_depth_link, origin xyz=0 0 0 rpy=${-pi/2} 0 ${-pi/2}
- added joint d455_back_joint: type fixed, parent middle_link, child d455_back_link, origin xyz=-0.155 0 0.42953 rpy=0 0 ${pi}, axis 0 0 1
- added joint d455_back_rgb_joint: type fixed, parent d455_back_link, child d455_back_rgb_link, origin xyz=0 0 0 rpy=${-pi/2} 0 ${-pi/2}
- added joint d455_front_depth_joint: type fixed, parent d455_front_link, child d455_front_depth_link, origin xyz=0 0 0 rpy=${-pi/2} 0 ${-pi/2}
- added joint d455_front_joint: type fixed, parent middle_link, child d455_front_link, origin xyz=0.18939 0.16173 0.428 rpy=${pi} 0.523599 0, axis 0 0 1
- added joint d455_front_rgb_joint: type fixed, parent d455_front_link, child d455_front_rgb_link, origin xyz=0 0 0 rpy=${-pi/2} 0 ${-pi/2}
- added joint left_back_rev: type continuous, parent base_link, child left_back, origin xyz=-0.2008 0.305 0.03 rpy=0 0 0, axis 0 1 0
- added joint left_front_rev: type continuous, parent base_link, child left_front, origin xyz=0.0532 0.305 0.03 rpy=0 0 0, axis 0 1 0
- added joint mid_joint: type fixed, parent base_link, child middle_link, origin xyz=0.0 0 0.15 rpy=0 0 0
- added joint right_back_rev: type continuous, parent base_link, child right_back, origin xyz=-0.2008 -0.305 0.03 rpy=0 0 0, axis 0 1 0
- added joint right_front_rev: type continuous, parent base_link, child right_front, origin xyz=0.0532 -0.305 0.03 rpy=0 0 0, axis 0 1 0

Commit message: fix lidar stuff

File: lunabot_description/urdf/mini_bot.xacro.urdf (robot description, URDF)
Before this commit: robot mini_bot, 14 links, 13 joints
Joints:
- joint lidar_mid_joint: origin xyz=0.18939 -0.51 0.44 rpy=0 ${-pi/2} 0 -> xyz=0.16939 -0.051 0.428 rpy=0 ${-pi/2} ${pi}; parent base_link -> middle_link

Commit message: Add minibot to the sim

File: lunabot_description/urdf/mini_bot.xacro.urdf (robot description, URDF)
Before this commit: robot mini_bot, 14 links, 13 joints
Links:
- removed link d455_back_depth_link
- removed link d455_back_rgb_link
- removed link d455_front_depth_link
- removed link d455_front_rgb_link
- added link d455_back_sim_link
- added link d455_front_sim_link
- link d455_back_link: mass 0.035 -> None; geometry visual box size=0.03 0.1 0.03
- link d455_front_link: mass 0.035 -> None; geometry visual box size=0.03 0.1 0.03
- link left_back: mass 5.0 -> None; geometry visual cylinder length=0.09 radius=0.03
- link left_front: mass 5.0 -> None; geometry visual cylinder length=0.09 radius=0.03
- link middle_link: mass 50.0 -> None; geometry visual box size=0.355 0.43 0.1
- link right_back: mass 5.0 -> None; geometry visual cylinder length=0.09 radius=0.03
- link right_front: mass 5.0 -> None; geometry visual cylinder length=0.09 radius=0.03
Joints:
- removed joint d455_back_depth_joint
- removed joint d455_back_rgb_joint
- removed joint d455_front_depth_joint
- removed joint d455_front_rgb_joint
- added joint d455_back_sim_joint: type fixed, parent d455_back_link, child d455_back_sim_link, origin xyz=0 0 0 rpy=${pi/2} 0 ${pi/2}
- added joint d455_front_sim_joint: type fixed, parent d455_front_link, child d455_front_sim_link, origin xyz=0 0 0 rpy=${pi/2} 0 ${pi/2}
