Commit message: sim and description: share robot constants between both representations
todo: fix xacro recompilation when a constant changes

File: lunabot_description/urdf/main_bot.xacro.urdf (robot description, URDF)
Before this commit: robot main_bot, 15 links, 14 joints
Links:
- link d455_back_link: geometry visual box size=${camera_dim_x} ${camera_dim_y} ${camera_dim_z}
- link d455_front_link: geometry visual box size=${camera_dim_x} ${camera_dim_y} ${camera_dim_z}
- link deposition_apriltag_link: geometry visual box size=${dep_apriltag_size} ${dep_apriltag_size} 0.001
- link deposition_apriltag_small_link: geometry visual box size=${dep_apriltag_small_size} ${dep_apriltag_small_size} 0.001
- link excavation: geometry visual box size=${exc_dim_x} ${exc_dim_y} ${exc_dim_z}
- link left_back: geometry visual cylinder length=${wheel_width} radius=${wheel_radius}
- link left_front: geometry visual cylinder length=${wheel_width} radius=${wheel_radius}
- link middle_link: geometry visual box size=${body_dim_x} ${body_dim_y} ${body_dim_z}
- link right_back: geometry visual cylinder length=${wheel_width} radius=${wheel_radius}
- link right_front: geometry visual cylinder length=${wheel_width} radius=${wheel_radius}
Joints:
- joint d455_back_joint: origin xyz=-0.44 0.02 0.63 rpy=${pi} 0.7 ${pi} -> xyz=${cam_back_x} ${cam_back_y} ${cam_back_z} rpy=${pi} ${cam_back_pitch} ${pi}
- joint d455_front_joint: origin xyz=0.3 0.0 -0.15 rpy=0 ${-0.663 + pi} 0 -> xyz=${cam_front_x} ${cam_front_y} ${cam_front_z} rpy=0 ${cam_front_pitch + pi} 0
- joint deposition_apriltag_joint: origin xyz=-0.42 -0.02 0.51 rpy=0.0 -0.35 3.14 -> xyz=${dep_apriltag_pos_x} ${dep_apriltag_pos_y} ${dep_apriltag_pos_z} rpy=0.0 ${dep_apriltag_pitch} ${pi}
- joint deposition_apriltag_optical_joint: origin xyz=0.0 0.0 0.0 rpy=1.57 0.0 1.57 -> xyz=0.0 0.0 0.0 rpy=${pi/2} 0.0 ${pi/2}
- joint deposition_apriltag_small_joint: origin xyz=-0.42 0.09 0.51 rpy=0.0 -0.35 3.14 -> xyz=${dep_apriltag_pos_x} ${dep_apriltag_small_pos_y} ${dep_apriltag_pos_z} rpy=0.0 ${dep_apriltag_pitch} ${pi}
- joint deposition_apriltag_small_optical_joint: origin xyz=0.0 0.0 0.0 rpy=1.57 0.0 1.57 -> xyz=0.0 0.0 0.0 rpy=${pi/2} 0.0 ${pi/2}
- joint excavation_joint: origin xyz=0.4 0 0.2 rpy=0 -2.0944 0 -> xyz=${exc_pos_x} 0 ${exc_pos_z} rpy=0 ${exc_pitch} 0; parent middle_link -> base_link
- joint left_back_rev: origin xyz=-0.228 0.254 0.178 rpy=0 0 0 -> xyz=-${back_wheel_pos_x} ${wheel_pos_y} ${wheel_pos_z} rpy=0 0 0
- joint left_front_rev: origin xyz=0.3302 0.254 0.178 rpy=0 0 0 -> xyz=${wheel_pos_x} ${wheel_pos_y} ${wheel_pos_z} rpy=0 0 0
- joint mid_joint: origin xyz=0.0 0 0.3 rpy=0 0 0 -> xyz=0.0 0 ${body_pos_z} rpy=0 0 0
- joint right_back_rev: origin xyz=-0.228 -0.254 0.178 rpy=0 0 0 -> xyz=-${back_wheel_pos_x} -${wheel_pos_y} ${wheel_pos_z} rpy=0 0 0
- joint right_front_rev: origin xyz=0.3302 -0.254 0.178 rpy=0 0 0 -> xyz=${wheel_pos_x} -${wheel_pos_y} ${wheel_pos_z} rpy=0 0 0

File: lunabot_description/urdf/mini_bot.xacro.urdf (robot description, URDF)
Before this commit: robot mini_bot, 12 links, 11 joints
Links:
- link d455_back_link: geometry visual box size=${camera_dim_x} ${camera_dim_y} ${camera_dim_z}
- link d455_front_link: geometry visual box size=${camera_dim_x} ${camera_dim_y} ${camera_dim_z}
- link left_back: geometry visual cylinder length=${wheel_width} radius=${wheel_radius}
- link left_front: geometry visual cylinder length=${wheel_width} radius=${wheel_radius}
- link middle_link: geometry visual box size=${body_dim_x} ${body_dim_y} ${body_dim_z}
- link right_back: geometry visual cylinder length=${wheel_width} radius=${wheel_radius}
- link right_front: geometry visual cylinder length=${wheel_width} radius=${wheel_radius}
Joints:
- joint d455_back_joint: origin xyz=-0.155 0 0.51 rpy=0 0 ${pi} -> xyz=${cam_back_x} ${cam_back_y} ${cam_back_z} rpy=0 0 ${pi}
- joint d455_front_joint: origin xyz=0.18939 0.16173 0.52 rpy=0 0.523599 0 -> xyz=${cam_front_x} ${cam_front_y} ${cam_front_z} rpy=0 ${cam_front_pitch} 0
- joint left_back_rev: origin xyz=-0.2008 0.305 0.03 rpy=0 0 0 -> xyz=-${back_wheel_pos_x} ${wheel_pos_y} ${wheel_pos_z} rpy=0 0 0
- joint left_front_rev: origin xyz=0.0532 0.305 0.03 rpy=0 0 0 -> xyz=${wheel_pos_x} ${wheel_pos_y} ${wheel_pos_z} rpy=0 0 0
- joint lidar_joint: origin xyz=0 0 0 rpy=0 0 ${pi*0.375} -> xyz=0 0 0 rpy=0 0 ${lidar_yaw}
- joint lidar_mid_joint: origin xyz=0.16939 -0.051 0.428 rpy=0 ${-pi/2} ${pi} -> xyz=${lidar_x} ${lidar_y} ${lidar_z} rpy=0 ${-pi/2} ${pi}
- joint mid_joint: origin xyz=0.0 0 0.15 rpy=0 0 0 -> xyz=0.0 0 ${body_pos_z} rpy=0 0 0
- joint right_back_rev: origin xyz=-0.2008 -0.305 0.03 rpy=0 0 0 -> xyz=-${back_wheel_pos_x} -${wheel_pos_y} ${wheel_pos_z} rpy=0 0 0
- joint right_front_rev: origin xyz=0.0532 -0.305 0.03 rpy=0 0 0 -> xyz=${wheel_pos_x} -${wheel_pos_y} ${wheel_pos_z} rpy=0 0 0
